Commit message: expé aujourd'hui

File: models/human_urdf/urdf/human.urdf (robot description, URDF)
Before this commit: robot human_5dof, 8 links, 7 joints
Joints:
- joint elbow_Z: origin xyz=0.262 0.0 0.0 rpy=0 -0 0 -> xyz=0.29 0.0 0.0 rpy=0 -0 0
- joint hand_fixed: origin xyz=0.273 0.0 0.0 rpy=0 -0 0 -> xyz=0.24 0.0 0.0 rpy=0 -0 0
- joint knee_Z: origin xyz=0.418 0.0 0.0 rpy=0 -0 0 -> xyz=0.38 0.0 0.0 rpy=0 -0 0
- joint lumbar_Z: origin xyz=0.417 0.0 0.0 rpy=0 -0 0 -> xyz=0.48 0.0 0.0 rpy=0 -0 0
- joint shoulder_Z: origin xyz=0.46 0.0 0.0 rpy=0 -0 0 -> xyz=0.45 0.0 0.0 rpy=0 -0 0
- joint world_to_human: origin xyz=0.0 0.0 0.0 rpy=1.57 -0 1.57 -> xyz=0. 0. 0. rpy=1.57 -0 -1.57

Commit message: adds human wb model

File: models/human_urdf/urdf/human.urdf (robot description, URDF)
Before this commit: robot human_5dof, 8 links, 7 joints
Links:
- removed link foot
- removed link hand
- removed link lowerarm
- removed link lowerleg
- removed link trunk
- removed link upperarm
- removed link upperleg
- added link left_clavicle, mass 0.15600
- added link left_foot, mass 1.13208; visual mesh filename=package://human_urdf/meshes/foot_mesh.STL scale=0.0060 0.0060 0.0060
- added link left_foot_virtual
- added link left_hand, mass 0.56604; visual mesh filename=package://human_urdf/meshes/hand_mesh.STL scale=0.0060 0.0060 0.0060
- added link left_hand_virtual
- added link left_lowerarm, mass 1.60378; visual mesh filename=package://human_urdf/meshes/lowerarm_mesh.STL scale=0.0060 0.0060 0.0060
- added link left_lowerarm_virtual; visual mesh filename=package://human_urdf/meshes/elbow_mesh.STL scale=0.0055 0.0055 0.0055
- added link left_lowerleg, mass 4.52832; visual mesh filename=package://human_urdf/meshes/lowerleg_mesh.STL scale=0.0063 0.0065 0.007
- added link left_upperarm, mass 2.26416; visual mesh filename=package://human_urdf/meshes/upperarm_mesh.STL scale=0.0063 0.0060 0.007
- added link left_upperarm_virtual; visual mesh filename=package://human_urdf/meshes/shoulder_mesh.STL scale=0.0055 0.0055 0.0055
- added link left_upperarm_virtual_2
- added link left_upperleg, mass 11.6038; visual mesh filename=package://human_urdf/meshes/upperleg_mesh.STL scale=0.0063 0.0065 0.007
- added link left_upperleg_virtual
- added link left_upperleg_virtual_2; visual mesh filename=package://human_urdf/meshes/knee_mesh.STL scale=0.006 0.006 0.006
- added link middle_abdomen, mass 2.73586; visual mesh filename=package://human_urdf/meshes/abdomen_mesh.STL scale=0.0055 0.0055 0.0055
- added link middle_abdomen_virtual
- added link middle_head, mass 6.32078; visual mesh filename=package://human_urdf/meshes/head_mesh.STL scale=0.0055 0.0055 0.0055
- added link middle_head_virtual; visual mesh filename=package://human_urdf/meshes/neck_mesh.STL scale=0.005 0.005 0.005
- added link middle_head_virtual_2
- added link middle_pelvis, mass 13.3963; visual mesh filename=package://human_urdf/meshes/pelvis_mesh.STL scale=0.006 0.0055 0.0055
- added link middle_thorax, mass 28.6794; visual mesh filename=package://human_urdf/meshes/torso_mesh.STL scale=0.0065 0.0065 0.0065
- added link middle_thorax_virtual
- added link middle_thorax_virtual_2
- added link right_clavicle, mass 0.15600
- added link right_foot, mass 1.13208; visual mesh filename=package://human_urdf/meshes/foot_mesh.STL scale=0.0060 0.0060 0.0060
- added link right_foot_virtual
- added link right_hand, mass 0.56604; visual mesh filename=package://human_urdf/meshes/hand_mesh.STL scale=0.0060 0.0060 0.0060
- added link right_hand_virtual
- added link right_lowerarm, mass 1.60378; visual mesh filename=package://human_urdf/meshes/lowerarm_mesh.STL scale=0.0060 0.0060 0.0060
- added link right_lowerarm_virtual; visual mesh filename=package://human_urdf/meshes/elbow_mesh.STL scale=0.0055 0.0055 0.0055
- added link right_lowerleg, mass 4.52832; visual mesh filename=package://human_urdf/meshes/lowerleg_mesh.STL scale=0.0063 0.0065 0.007
- added link right_upperarm, mass 2.26416; visual mesh filename=package://human_urdf/meshes/upperarm_mesh.STL scale=0.0063 0.0060 0.007
- added link right_upperarm_virtual; visual mesh filename=package://human_urdf/meshes/shoulder_mesh.STL scale=0.0055 0.0055 0.0055
- added link right_upperarm_virtual_2
- added link right_upperleg, mass 11.6038; visual mesh filename=package://human_urdf/meshes/upperleg_mesh.STL scale=0.0063 0.0065 0.007
- added link right_upperleg_virtual
- added link right_upperleg_virtual_2; visual mesh filename=package://human_urdf/meshes/knee_mesh.STL scale=0.006 0.006 0.006
Joints:
- removed joint ankle_Z
- removed joint elbow_Z
- removed joint hand_fixed
- removed joint knee_Z
- removed joint lumbar_Z
- removed joint shoulder_Z
- added joint left_ankle_X: type revolute, parent left_foot_virtual, child left_foot, origin xyz=0 0 0 rpy=0 -0 0, axis -1 0 0, limit lower=0 upper=0.785398 effort=0 velocity=0
- added joint left_ankle_Z: type revolute, parent left_lowerleg, child left_foot_virtual, origin xyz=0 -0.42805 0 rpy=0 -0 0, axis 0 0 1, limit lower=-0.392699 upper=1.0472 effort=0 velocity=0
- added joint left_clavicle_joint_X: type revolute, parent middle_thorax, child left_clavicle, origin xyz=0 0.330225 0 rpy=0 -0 0, axis 1 0 0, limit lower=-1.0472 upper=0.314159 effort=0 velocity=0
- added joint left_elbow_Y: type revolute, parent left_lowerarm_virtual, child left_lowerarm, origin xyz=0 0 0 rpy=0 -0 0, axis 0 -1 0, limit lower=-1.5708 upper=1.5708 effort=0 velocity=0
- added joint left_elbow_Z: type revolute, parent left_upperarm, child left_lowerarm_virtual, origin xyz=0 -0.2737 0 rpy=0 -0 0, axis 0 0 1, limit lower=0 upper=2.74889 effort=0 velocity=0
- added joint left_hip_X: type revolute, parent left_upperleg_virtual, child left_upperleg_virtual_2, origin xyz=0 0 0 rpy=0 -0 0, axis 1 0 0, limit lower=-0.392699 upper=1.5708 effort=0 velocity=0
- added joint left_hip_Y: type revolute, parent left_upperleg_virtual_2, child left_upperleg, origin xyz=0 0 0 rpy=0 -0 0, axis 0 1 0, limit lower=-1.5708 upper=1.5708 effort=0 velocity=0
- added joint left_hip_Z: type revolute, parent middle_pelvis, child left_upperleg_virtual, origin xyz=0.053375 -0.0749 -0.079975 rpy=0 -0 0, axis 0 0 1, limit lower=-0.785398 upper=3.14159 effort=0 velocity=0
- added joint left_knee: type revolute, parent left_upperleg, child left_lowerleg, origin xyz=0 -0.427 0 rpy=0 -0 0, axis 0 0 -1, limit lower=0 upper=2.74889 effort=0 velocity=0
- added joint left_shoulder_X: type revolute, parent left_upperarm_virtual, child left_upperarm_virtual_2, origin xyz=0 0 0 rpy=0 -0 0, axis 1 0 0, limit lower=-3.14159 upper=1.0472 effort=0 velocity=0
- added joint left_shoulder_Y: type revolute, parent left_upperarm_virtual_2, child left_upperarm, origin xyz=0 0 0 rpy=0 -0 0, axis 0 1 0, limit lower=-1.5708 upper=3.14159 effort=0 velocity=0
- added joint left_shoulder_Z: type revolute, parent left_clavicle, child left_upperarm_virtual, origin xyz=0.00805 -0.0728 -0.2037 rpy=0 -0 0, axis 0 0 1, limit lower=-2.0944 upper=0.392699 effort=0 velocity=0
- added joint left_wrist_X: type revolute, parent left_hand_virtual, child left_hand, origin xyz=0 0 0 rpy=0 -0 0, axis -1 0 0, limit lower=-0.785398 upper=0.785398 effort=0 velocity=0
- added joint left_wrist_Z: type revolute, parent left_lowerarm, child left_hand_virtual, origin xyz=0 -0.27965 0 rpy=0 -0 0, axis 0 0 1, limit lower=-1.5708 upper=1.5708 effort=0 velocity=0
- added joint middle_cervical_X: type revolute, parent middle_head_virtual, child middle_head_virtual_2, origin xyz=0 0 0 rpy=0 -0 0, axis 1 0 0, limit lower=-1.0472 upper=1.0472 effort=0 velocity=0
- added joint middle_cervical_Y: type revolute, parent middle_head_virtual_2, child middle_head, origin xyz=0 0 0 rpy=0 -0 0, axis 0 1 0, limit lower=-1.5708 upper=1.5708 effort=0 velocity=0
- added joint middle_cervical_Z: type revolute, parent middle_thorax, child middle_head_virtual, origin xyz=0 0.330225 0 rpy=0 -0 0, axis 0 0 -1, limit lower=-1.5708 upper=1.5708 effort=0 velocity=0
- added joint middle_lumbar_X: type revolute, parent middle_abdomen_virtual, child middle_abdomen, origin xyz=0 0 0 rpy=0 -0 0, axis 1 0 0, limit lower=-0.785398 upper=0.785398 effort=0 velocity=0
- added joint middle_lumbar_Z: type revolute, parent middle_pelvis, child middle_abdomen_virtual, origin xyz=0 0 0 rpy=0 -0 0, axis 0 0 -1, limit lower=-3.14159 upper=0.785398 effort=0 velocity=0
- added joint middle_thoracic_X: type revolute, parent middle_thorax_virtual, child middle_thorax_virtual_2, origin xyz=0 0 0 rpy=0 -0 0, axis 1 0 0, limit lower=-1.0472 upper=1.0472 effort=0 velocity=0
- added joint middle_thoracic_Y: type revolute, parent middle_thorax_virtual_2, child middle_thorax, origin xyz=0 0 0 rpy=0 -0 0, axis 0 1 0, limit lower=-1.0472 upper=1.0472 effort=0 velocity=0
- added joint middle_thoracic_Z: type revolute, parent middle_abdomen, child middle_thorax_virtual, origin xyz=0 0.149275 0 rpy=0 -0 0, axis 0 0 -1, limit lower=-1.0472 upper=0.392699 effort=0 velocity=0
- added joint right_ankle_X: type revolute, parent right_foot_virtual, child right_foot, origin xyz=0 0 0 rpy=0 -0 0, axis 1 0 0, limit lower=0 upper=0.785398 effort=0 velocity=0
- added joint right_ankle_Z: type revolute, parent right_lowerleg, child right_foot_virtual, origin xyz=0 -0.42805 0 rpy=0 -0 0, axis 0 0 1, limit lower=-1.0472 upper=0.392699 effort=0 velocity=0
- added joint right_clavicle_joint_X: type revolute, parent middle_thorax, child right_clavicle, origin xyz=0 0.330225 0 rpy=0 -0 0, axis -1 0 0, limit lower=-0.392699 upper=1.0472 effort=0 velocity=0
- added joint right_elbow_Y: type revolute, parent right_lowerarm_virtual, child right_lowerarm, origin xyz=0 0 0 rpy=0 -0 0, axis 0 1 0, limit lower=-1.5708 upper=1.5708 effort=0 velocity=0
- added joint right_elbow_Z: type revolute, parent right_upperarm, child right_lowerarm_virtual, origin xyz=0 -0.2737 0 rpy=0 -0 0, axis 0 0 1, limit lower=0 upper=2.74889 effort=0 velocity=0
- added joint right_hip_X: type revolute, parent right_upperleg_virtual, child right_upperleg_virtual_2, origin xyz=0 0 0 rpy=0 -0 0, axis -1 0 0, limit lower=-0.392699 upper=1.5708 effort=0 velocity=0
- added joint right_hip_Y: type revolute, parent right_upperleg_virtual_2, child right_upperleg, origin xyz=0 0 0 rpy=0 -0 0, axis 0 -1 0, limit lower=-1.5708 upper=1.5708 effort=0 velocity=0
- added joint right_hip_Z: type revolute, parent middle_pelvis, child right_upperleg_virtual, origin xyz=0.053375 -0.0749 0.079975 rpy=0 -0 0, axis 0 0 1, limit lower=-0.785398 upper=3.14159 effort=0 velocity=0
- added joint right_knee: type revolute, parent right_upperleg, child right_lowerleg, origin xyz=0 -0.427 0 rpy=0 -0 0, axis 0 0 -1, limit lower=0 upper=2.74889 effort=0 velocity=0
- added joint right_shoulder_X: type revolute, parent right_upperarm_virtual, child right_upperarm_virtual_2, origin xyz=0 0 0 rpy=0 -0 0, axis -1 0 0, limit lower=-3.14159 upper=1.0472 effort=0 velocity=0
- added joint right_shoulder_Y: type revolute, parent right_upperarm_virtual_2, child right_upperarm, origin xyz=0 0 0 rpy=0 -0 0, axis 0 -1 0, limit lower=-1.5708 upper=3.14159 effort=0 velocity=0
- added joint right_shoulder_Z: type revolute, parent right_clavicle, child right_upperarm_virtual, origin xyz=0.00805 -0.0728 0.2037 rpy=0 -0 0, axis 0 0 1, limit lower=-2.0944 upper=0.392699 effort=0 velocity=0
- added joint right_wrist_X: type revolute, parent right_hand_virtual, child right_hand, origin xyz=0 0 0 rpy=0 -0 0, axis 1 0 0, limit lower=-0.785398 upper=0.785398 effort=0 velocity=0
- added joint right_wrist_Z: type revolute, parent right_lowerarm, child right_hand_virtual, origin xyz=0 -0.27965 0 rpy=0 -0 0, axis 0 0 1, limit lower=-1.5708 upper=1.5708 effort=0 velocity=0
- joint world_to_human: child foot -> middle_pelvis; origin xyz=0. 0. 0. rpy=1.57 -0 -1.57 -> xyz=0. 0. 0. rpy=1.57 -0 0

Commit message: human model generation both urdf or pinocchio wise

File: models/human_urdf/urdf/human.urdf (robot description, URDF)
Before this commit: robot human_36dof_ISB_model, 38 links, 37 joints
Joints:
- removed joint left_knee
- removed joint right_knee
- added joint left_knee_Z: type revolute, parent left_upperleg, child left_lowerleg, origin xyz=0 -0.427 0 rpy=0 -0 0, axis 0 0 -1, limit lower=0 upper=2.74889 effort=0 velocity=0
- added joint right_knee_Z: type revolute, parent right_upperleg, child right_lowerleg, origin xyz=0 -0.427 0 rpy=0 -0 0, axis 0 0 -1, limit lower=0 upper=2.74889 effort=0 velocity=0

Commit message: add urdf but not sure if pin model and urdf model are the same

File: models/human_urdf/urdf/human.urdf (robot description, URDF)
Before this commit: robot human_36dof_ISB_model, 38 links, 37 joints
Links:
- removed link left_clavicle
- removed link left_foot
- removed link left_foot_virtual
- removed link left_hand
- removed link left_hand_virtual
- removed link left_lowerarm
- removed link left_lowerarm_virtual
- removed link left_lowerleg
- removed link left_upperarm
- removed link left_upperarm_virtual
- removed link left_upperarm_virtual_2
- removed link left_upperleg
- removed link left_upperleg_virtual
- removed link left_upperleg_virtual_2
- removed link middle_abdomen
- removed link middle_abdomen_virtual
- removed link middle_head
- removed link middle_head_virtual
- removed link middle_head_virtual_2
- removed link middle_pelvis
- removed link middle_thorax
- removed link middle_thorax_virtual
- removed link middle_thorax_virtual_2
- removed link right_clavicle
- removed link right_foot
- removed link right_foot_virtual
- removed link right_hand
- removed link right_hand_virtual
- removed link right_lowerarm
- removed link right_lowerarm_virtual
- removed link right_lowerleg
- removed link right_upperarm
- removed link right_upperarm_virtual
- removed link right_upperarm_virtual_2
- removed link right_upperleg
- removed link right_upperleg_virtual
- removed link right_upperleg_virtual_2
- removed link world
- added link footL, mass 1.13208; visual mesh filename=package://human_urdf/meshes/foot_mesh.STL scale=0.0060 0.0060 0.0060
- added link footR, mass 1.13208; visual mesh filename=package://human_urdf/meshes/foot_mesh.STL scale=0.0060 0.0060 0.0060
- added link lowerarmL, mass 1.60378; visual mesh filename=package://human_urdf/meshes/lowerarm_mesh.STL scale=0.0060 0.0060 0.0060
- added link lowerarmR, mass 1.60378; visual mesh filename=package://human_urdf/meshes/lowerarm_mesh.STL scale=0.0060 0.0060 0.0060
- added link lowerarm_z; visual mesh filename=package://human_urdf/meshes/elbow_mesh.STL scale=0.0055 0.0055 0.0055
- added link lowerarm_z_L; visual mesh filename=package://human_urdf/meshes/elbow_mesh.STL scale=0.0055 0.0055 0.0055
- added link pelvis, mass 13.3963; visual mesh filename=package://human_urdf/meshes/pelvis_mesh.STL scale=0.006 0.0055 0.0055
- added link shankL, mass 4.52832; visual mesh filename=package://human_urdf/meshes/lowerleg_mesh.STL scale=0.0063 0.0065 0.007
- added link shankR, mass 4.52832; visual mesh filename=package://human_urdf/meshes/lowerleg_mesh.STL scale=0.0063 0.0065 0.007
- added link thighL, mass 11.6038; visual mesh filename=package://human_urdf/meshes/upperleg_mesh.STL scale=0.0063 0.0065 0.007
- added link thighR, mass 11.6038; visual mesh filename=package://human_urdf/meshes/upperleg_mesh.STL scale=0.0063 0.0065 0.007
- added link thigh_x; visual mesh filename=package://human_urdf/meshes/knee_mesh.STL scale=0.006 0.006 0.006
- added link thigh_x_L; visual mesh filename=package://human_urdf/meshes/knee_mesh.STL scale=0.006 0.006 0.006
- added link thigh_z
- added link thigh_z_L
- added link torso, mass 28.6794; visual mesh filename=package://human_urdf/meshes/abdomen_mesh.STL scale=0.0055 0.0055 0.0055; visual mesh filename=package://human_urdf/meshes/torso_mesh.STL scale=0.0065 0.0065 0.0065
- added link torso_z
- added link upperarmL, mass 2.26416; visual mesh filename=package://human_urdf/meshes/upperarm_mesh.STL scale=0.0063 0.0060 0.007
- added link upperarmR, mass 2.26416; visual mesh filename=package://human_urdf/meshes/upperarm_mesh.STL scale=0.0063 0.0060 0.007
- added link upperarm_x_L
- added link upperarm_x_R
- added link upperarm_z_L; visual mesh filename=package://human_urdf/meshes/shoulder_mesh.STL scale=0.0055 0.0055 0.0055
- added link upperarm_z_R; visual mesh filename=package://human_urdf/meshes/shoulder_mesh.STL scale=0.0055 0.0055 0.0055
Joints:
- removed joint left_ankle_X
- removed joint left_clavicle_joint_X
- removed joint left_wrist_X
- removed joint left_wrist_Z
- removed joint middle_cervical_X
- removed joint middle_cervical_Y
- removed joint middle_cervical_Z
- removed joint middle_lumbar_X
- removed joint middle_thoracic_X
- removed joint middle_thoracic_Y
- removed joint middle_thoracic_Z
- removed joint right_ankle_X
- removed joint right_clavicle_joint_X
- removed joint right_wrist_X
- removed joint right_wrist_Z
- removed joint world_to_human
- added joint middle_lumbar_Y: type revolute, parent torso_z, child torso, origin xyz=0 0 0 rpy=0 -0 0, axis 1 0 0, limit lower=-0.785398 upper=0.785398 effort=0 velocity=0
- joint left_ankle_Z: child left_foot_virtual -> footL; parent left_lowerleg -> shankL
- joint left_elbow_Y: axis 0 -1 0 -> 0 1 0; child left_lowerarm -> lowerarmL; parent left_lowerarm_virtual -> lowerarm_z_L
- joint left_elbow_Z: child left_lowerarm_virtual -> lowerarm_z_L; parent left_upperarm -> upperarmL
- joint left_hip_X: child left_upperleg_virtual_2 -> thigh_x_L; parent left_upperleg_virtual -> thigh_z_L
- joint left_hip_Y: child left_upperleg -> thighL; parent left_upperleg_virtual_2 -> thigh_x_L
- joint left_hip_Z: child left_upperleg_virtual -> thigh_z_L; parent middle_pelvis -> pelvis
- joint left_knee_Z: axis 0 0 -1 -> 0 0 1; child left_lowerleg -> shankL; parent left_upperleg -> thighL
- joint left_shoulder_X: child left_upperarm_virtual_2 -> upperarm_x_L; parent left_upperarm_virtual -> upperarm_z_L
- joint left_shoulder_Y: child left_upperarm -> upperarmL; parent left_upperarm_virtual_2 -> upperarm_x_L
- joint left_shoulder_Z: child left_upperarm_virtual -> upperarm_z_L; origin xyz=0.00805 -0.0728 -0.2037 rpy=0 -0 0 -> xyz=0.00805 0.4067 -0.2037 rpy=0 -0 0; parent left_clavicle -> torso
- joint middle_lumbar_Z: axis 0 0 -1 -> 0 0 1; child middle_abdomen_virtual -> torso_z; parent middle_pelvis -> pelvis
- joint right_ankle_Z: child right_foot_virtual -> footR; parent right_lowerleg -> shankR
- joint right_elbow_Y: child right_lowerarm -> lowerarmR; parent right_lowerarm_virtual -> lowerarm_z
- joint right_elbow_Z: child right_lowerarm_virtual -> lowerarm_z; parent right_upperarm -> upperarmR
- joint right_hip_X: axis -1 0 0 -> 1 0 0; child right_upperleg_virtual_2 -> thigh_x; parent right_upperleg_virtual -> thigh_z
- joint right_hip_Y: axis 0 -1 0 -> 0 1 0; child right_upperleg -> thighR; parent right_upperleg_virtual_2 -> thigh_x
- joint right_hip_Z: child right_upperleg_virtual -> thigh_z; parent middle_pelvis -> pelvis
- joint right_knee_Z: axis 0 0 -1 -> 0 0 1; child right_lowerleg -> shankR; parent right_upperleg -> thighR
- joint right_shoulder_X: axis -1 0 0 -> 1 0 0; child right_upperarm_virtual_2 -> upperarm_x_R; parent right_upperarm_virtual -> upperarm_z_R
- joint right_shoulder_Y: axis 0 -1 0 -> 0 1 0; child right_upperarm -> upperarmR; parent right_upperarm_virtual_2 -> upperarm_x_R
- joint right_shoulder_Z: child right_upperarm_virtual -> upperarm_z_R; origin xyz=0.00805 -0.0728 0.2037 rpy=0 -0 0 -> xyz=0.00805 0.4067 0.2037 rpy=0 -0 0; parent right_clavicle -> torso
