Commit message: ros layer for visu in rviz

File: urdf/human.urdf.xacro (robot description, xacro)
@@ -1,3 +1,10 @@
-<robot name="human_wb_ISB_model">
+<?xml version="1.0" encoding="utf-8"?>
+<robot xmlns:xacro="http://wiki.ros.org/xacro">
+    <joint name="world_to_human" type="fixed">
+      <origin rpy="1.57 -0 0" xyz="0. 0. 0."/>
+      <axis xyz="0 0 1"/>
+      <parent link="world"/>
+      <child link="pelvis"/>
+    </joint>
     <material name="body_color">
         <texture />
@@ -13,5 +20,5 @@
 	        <origin xyz="-0.08 -0.13 0.125" rpy="0 1.57 0" />
             <geometry>
-		        <mesh filename="package://human_urdf/meshes/pelvis_mesh.STL" scale="0.006 0.0055 0.0055"/>
+		        <mesh filename="package://rt_cosmik/meshes/pelvis_mesh.STL" scale="0.006 0.0055 0.0055"/>
             </geometry>
             <material name="body_color">
@@ -45,5 +52,5 @@
             <origin xyz="-0.05 0.05 -0.085" rpy="0 -0 0" />
             <geometry>
-		        <mesh filename="package://human_urdf/meshes/abdomen_mesh.STL" scale="0.0055 0.0055 0.0055"/>
+		        <mesh filename="package://rt_cosmik/meshes/abdomen_mesh.STL" scale="0.0055 0.0055 0.0055"/>
                 <!--<box size="0.15 0.161217 0.198658" />-->
             </geometry>
@@ -57,5 +64,5 @@
             <geometry>
 		        <!--<box size="0.15 0.356643 0.329994" />-->
-		        <mesh filename="package://human_urdf/meshes/torso_mesh.STL" scale="0.0065 0.0065 0.0065"/>
+		        <mesh filename="package://rt_cosmik/meshes/torso_mesh.STL" scale="0.0065 0.0065 0.0065"/>
             </geometry>
             <material name="body_color">
@@ -76,5 +83,5 @@
 	        <origin xyz="-0.15 -0.04 -0.05" rpy="0 0 0" />
             <geometry>
-		        <mesh filename="package://human_urdf/meshes/shoulder_mesh.STL" scale="0.0055 0.0055 0.0055"/>
+		        <mesh filename="package://rt_cosmik/meshes/shoulder_mesh.STL" scale="0.0055 0.0055 0.0055"/>
             </geometry>
             <material name="body_color">
@@ -108,5 +115,5 @@
             <origin xyz="-0.065 -0.27 0.18" rpy="0.0 1.57 0" />
             <geometry>
-                <mesh filename="package://human_urdf/meshes/upperarm_mesh.STL" scale="0.0063 0.0060 0.007"/>
+                <mesh filename="package://rt_cosmik/meshes/upperarm_mesh.STL" scale="0.0063 0.0060 0.007"/>
             </geometry>
             <material name="body_color">
@@ -127,5 +134,5 @@
 	        <origin xyz="-0.15 -0.04 -0.035" rpy="0 0 0" />
             <geometry>
-		        <mesh filename="package://human_urdf/meshes/elbow_mesh.STL" scale="0.0055 0.0055 0.0055"/>
+		        <mesh filename="package://rt_cosmik/meshes/elbow_mesh.STL" scale="0.0055 0.0055 0.0055"/>
             </geometry>
             <material name="body_color">
@@ -151,5 +158,5 @@
             <origin xyz="0.052 -0.26 -0.17" rpy="0.0 -1.57 0" />
             <geometry>
-                <mesh filename="package://human_urdf/meshes/lowerarm_mesh.STL" scale="0.0060 0.0060 0.0060"/>
+                <mesh filename="package://rt_cosmik/meshes/lowerarm_mesh.STL" scale="0.0060 0.0060 0.0060"/>
             </geometry>
             <material name="body_color">
@@ -170,5 +177,5 @@
 	        <origin xyz="-0.16 -0.045 -0.045" rpy="0 0 0" />
             <geometry>
-		        <mesh filename="package://human_urdf/meshes/shoulder_mesh.STL" scale="0.0055 0.0055 0.0055"/>
+		        <mesh filename="package://rt_cosmik/meshes/shoulder_mesh.STL" scale="0.0055 0.0055 0.0055"/>
             </geometry>
             <material name="body_color">
@@ -202,5 +209,5 @@
             <origin xyz="-0.065 -0.27 0.18" rpy="0.0 1.57 0" />
             <geometry>
-                <mesh filename="package://human_urdf/meshes/upperarm_mesh.STL" scale="0.0063 0.0060 0.007"/>
+                <mesh filename="package://rt_cosmik/meshes/upperarm_mesh.STL" scale="0.0063 0.0060 0.007"/>
             </geometry>
             <material name="body_color"/>
@@ -218,5 +225,5 @@
 	        <origin xyz="-0.15 -0.04 -0.035" rpy="0 0 0" />
             <geometry>
-		        <mesh filename="package://human_urdf/meshes/elbow_mesh.STL" scale="0.0055 0.0055 0.0055"/>
+		        <mesh filename="package://rt_cosmik/meshes/elbow_mesh.STL" scale="0.0055 0.0055 0.0055"/>
             </geometry>
             <material name="body_color">
@@ -242,5 +249,5 @@
             <origin xyz="0.052 -0.26 -0.17" rpy="0.0 -1.57 0" />
             <geometry>
-                <mesh filename="package://human_urdf/meshes/lowerarm_mesh.STL" scale="0.0060 0.0060 0.0060"/>
+                <mesh filename="package://rt_cosmik/meshes/lowerarm_mesh.STL" scale="0.0060 0.0060 0.0060"/>
             </geometry>
             <material name="body_color">
@@ -269,5 +276,5 @@
             <origin xyz="-0.04 -0.48 0.07" rpy="0.0 1.57 0" />
             <geometry>
-                <mesh filename="package://human_urdf/meshes/knee_mesh.STL" scale="0.006 0.006 0.006"/>
+                <mesh filename="package://rt_cosmik/meshes/knee_mesh.STL" scale="0.006 0.006 0.006"/>
             </geometry>
             <material name="body_color">
@@ -293,5 +300,5 @@
             <origin xyz="-0.1 -0.42 0.07" rpy="0.0 1.57 0" />
             <geometry>
-                <mesh filename="package://human_urdf/meshes/upperleg_mesh.STL" scale="0.0063 0.0065 0.007"/>
+                <mesh filename="package://rt_cosmik/meshes/upperleg_mesh.STL" scale="0.0063 0.0065 0.007"/>
             </geometry>
             <material name="body_color">
@@ -317,5 +324,5 @@
             <origin xyz="-0.06 -0.43 0.07" rpy="0.0 1.57 0" />
             <geometry>
-                <mesh filename="package://human_urdf/meshes/lowerleg_mesh.STL" scale="0.0063 0.0065 0.007"/>
+                <mesh filename="package://rt_cosmik/meshes/lowerleg_mesh.STL" scale="0.0063 0.0065 0.007"/>
             </geometry>
             <material name="body_color">
@@ -341,5 +348,5 @@
             <origin xyz="-0.05 -0.055 0.065" rpy="0 1.57 0" />
             <geometry>
-		        <mesh filename="package://human_urdf/meshes/foot_mesh.STL" scale="0.0060 0.0060 0.0060"/>
+		        <mesh filename="package://rt_cosmik/meshes/foot_mesh.STL" scale="0.0060 0.0060 0.0060"/>
                 <!--<box size="0.03 0.085239 0.06" />-->
             </geometry>
@@ -369,5 +376,5 @@
             <origin xyz="-0.04 -0.48 0.080" rpy="0.0 1.57 0" />
             <geometry>
-                <mesh filename="package://human_urdf/meshes/knee_mesh.STL" scale="0.006 0.006 0.006"/>
+                <mesh filename="package://rt_cosmik/meshes/knee_mesh.STL" scale="0.006 0.006 0.006"/>
             </geometry>
             <material name="body_color">
@@ -393,5 +400,5 @@
             <origin xyz="-0.1 -0.42 0.085" rpy="0.0 1.57 0" />
             <geometry>
-                <mesh filename="package://human_urdf/meshes/upperleg_mesh.STL" scale="0.0063 0.0065 0.007"/>
+                <mesh filename="package://rt_cosmik/meshes/upperleg_mesh.STL" scale="0.0063 0.0065 0.007"/>
             </geometry>
             <material name="body_color">
@@ -417,5 +424,5 @@
             <origin xyz="-0.06 -0.43 0.08" rpy="0.0 1.57 0" />
             <geometry>
-                <mesh filename="package://human_urdf/meshes/lowerleg_mesh.STL" scale="0.0063 0.0065 0.007"/>
+                <mesh filename="package://rt_cosmik/meshes/lowerleg_mesh.STL" scale="0.0063 0.0065 0.007"/>
             </geometry>
             <material name="body_color">
@@ -441,5 +448,5 @@
             <origin xyz="-0.05 -0.055 0.075" rpy="0 1.57 0" />
             <geometry>
-		        <mesh filename="package://human_urdf/meshes/foot_mesh.STL" scale="0.0060 0.0060 0.0060"/>
+		        <mesh filename="package://rt_cosmik/meshes/foot_mesh.STL" scale="0.0060 0.0060 0.0060"/>
                 <!--<box size="0.03 0.085239 0.06" />-->
             </geometry>

File: urdf/human_5dof.urdf (robot description, URDF)
Before this commit: robot human_5dof, 8 links, 7 joints
Links:
- link foot: geometry visual mesh filename=package://rt_cosmik/meshes/foot_mesh.STL scale=0.0060 0.0060 0.0060; visual mesh filename=package://rt_cosmik/meshes/foot_mesh.STL scale=0.0060 0.0060 0.0060
- link hand: geometry visual mesh filename=package://rt_cosmik/meshes/hand_mesh.STL scale=0.0060 0.0060 0.0060; visual mesh filename=package://rt_cosmik/meshes/hand_mesh.STL scale=0.0060 0.0060 0.0060
- link lowerarm: geometry visual mesh filename=package://rt_cosmik/meshes/elbow_mesh.STL scale=0.0055 0.0055 0.0055; visual mesh filename=package://rt_cosmik/meshes/elbow_mesh.STL scale=0.0055 0.0055 0.0055
- link lowerleg: geometry visual mesh filename=package://rt_cosmik/meshes/lowerleg_mesh.STL scale=0.0063 0.0065 0.007; visual mesh filename=package://rt_cosmik/meshes/lowerleg_mesh.STL scale=0.0063 0.0065 0.007
- link trunk: geometry visual mesh filename=package://rt_cosmik/meshes/abdomen_mesh.STL scale=0.0055 0.0055 0.0055; visual mesh filename=package://rt_cosmik/meshes/head_mesh.STL scale=0.0055 0.0055 0.0055
- link upperarm: geometry visual mesh filename=package://rt_cosmik/meshes/shoulder_mesh.STL scale=0.0055 0.0055 0.0055; visual mesh filename=package://rt_cosmik/meshes/shoulder_mesh.STL scale=0.0055 0.0055 0.0055
- link upperleg: geometry visual mesh filename=package://rt_cosmik/meshes/knee_mesh.STL scale=0.006 0.006 0.006; visual mesh filename=package://rt_cosmik/meshes/knee_mesh.STL scale=0.006 0.006 0.006
