Commit message: work on ik for 5 dof model but still need to understand why it does not track

File: urdf/human_5dof.urdf (robot description, URDF)
Before this commit: robot human_5dof, 8 links, 7 joints
Joints:
- joint world_to_human: origin xyz=0. 0. 0. rpy=1.57 -0 -1.57 -> xyz=0.00056 -0.0133 0.1036 rpy=1.5478 0.1048 0.908

Commit message: setup expe

File: urdf/human_5dof.urdf (robot description, URDF)
Before this commit: robot human_5dof, 8 links, 7 joints
Joints:
- joint elbow_Z: origin xyz=0.29 0.0 0.0 rpy=0 -0 0 -> xyz=0.3328 0.0 0.0 rpy=0 -0 0
- joint hand_fixed: origin xyz=0.24 0.0 0.0 rpy=0 -0 0 -> xyz=0.2380 0.0 0.0 rpy=0 -0 0
- joint knee_Z: origin xyz=0.38 0.0 0.0 rpy=0 -0 0 -> xyz=0.3954 0.0 0.0 rpy=0 -0 0
- joint lumbar_Z: origin xyz=0.48 0.0 0.0 rpy=0 -0 0 -> xyz=0.4777 0.0 0.0 rpy=0 -0 0
- joint shoulder_Z: origin xyz=0.45 0.0 0.0 rpy=0 -0 0 -> xyz=0.4232 0.0 0.0 rpy=0 -0 0

Commit message: fix + calib

File: urdf/human_5dof.urdf (robot description, URDF)
Before this commit: robot human_5dof, 8 links, 7 joints
Joints:
- joint world_to_human: origin xyz=0.00056 -0.0133 0.1036 rpy=1.5478 0.1048 0.908 -> xyz=0.0287 0.004 0.0225 rpy=1.5647 0.0780 0.8973

Commit message: post expe of the day

File: urdf/human_5dof.urdf (robot description, URDF)
Before this commit: robot human_5dof, 8 links, 7 joints
Joints:
- joint elbow_Z: origin xyz=0.3328 0.0 0.0 rpy=0 -0 0 -> xyz=0.3369 0.0 0.0 rpy=0 -0 0
- joint hand_fixed: origin xyz=0.2380 0.0 0.0 rpy=0 -0 0 -> xyz=0.2327 0.0 0.0 rpy=0 -0 0
- joint knee_Z: origin xyz=0.3954 0.0 0.0 rpy=0 -0 0 -> xyz=0.3886 0.0 0.0 rpy=0 -0 0
- joint lumbar_Z: origin xyz=0.4777 0.0 0.0 rpy=0 -0 0 -> xyz=0.4909 0.0 0.0 rpy=0 -0 0
- joint shoulder_Z: origin xyz=0.4232 0.0 0.0 rpy=0 -0 0 -> xyz=0.4598 0.0 0.0 rpy=0 -0 0

Commit message: scaling maxime

File: urdf/human_5dof.urdf (robot description, URDF)
Before this commit: robot human_5dof, 8 links, 7 joints
Joints:
- joint elbow_Z: origin xyz=0.3369 0.0 0.0 rpy=0 -0 0 -> xyz=0.3150 0.0 0.0 rpy=0 -0 0
- joint hand_fixed: origin xyz=0.2327 0.0 0.0 rpy=0 -0 0 -> xyz=0.2358 0.0 0.0 rpy=0 -0 0
- joint knee_Z: origin xyz=0.3886 0.0 0.0 rpy=0 -0 0 -> xyz=0.3989 0.0 0.0 rpy=0 -0 0
- joint lumbar_Z: origin xyz=0.4909 0.0 0.0 rpy=0 -0 0 -> xyz=0.4812 0.0 0.0 rpy=0 -0 0
- joint shoulder_Z: origin xyz=0.4598 0.0 0.0 rpy=0 -0 0 -> xyz=0.4367 0.0 0.0 rpy=0 -0 0

Commit message: ajout des paramètres anthropométriques humains dans le fichier YAML

File: urdf/human_5dof.urdf (robot description, URDF)
Before this commit: robot human_5dof, 8 links, 7 joints
Joints:
- joint elbow_Z: origin xyz=0.3150 0.0 0.0 rpy=0 -0 0 -> xyz=0.33566674458246937 0 0 rpy=0 -0 0
- joint hand_fixed: origin xyz=0.2358 0.0 0.0 rpy=0 -0 0 -> xyz=0.23242554243018573 0 0 rpy=0 -0 0
- joint knee_Z: origin xyz=0.3989 0.0 0.0 rpy=0 -0 0 -> xyz=0.40155370945561 0 0 rpy=0 -0 0
- joint lumbar_Z: origin xyz=0.4812 0.0 0.0 rpy=0 -0 0 -> xyz=0.47648042433424215 0 0 rpy=0 -0 0
- joint shoulder_Z: origin xyz=0.4367 0.0 0.0 rpy=0 -0 0 -> xyz=0.4397691087116175 0 0 rpy=0 -0 0
- joint world_to_human: origin xyz=0.0287 0.004 0.0225 rpy=1.5647 0.0780 0.8973 -> xyz=0.02373367081544142 0.005079786187961677 0.010846197486314102 rpy=1.572570285861921 0.15063584360293358 0.9840076914665431

Commit message: change model bounds

File: urdf/human_5dof.urdf (robot description, URDF)
Before this commit: robot human_5dof, 8 links, 7 joints
Joints:
- joint ankle_Z: limit lower=-3.14 upper=3.14159 effort=500.0 velocity=200.0 -> lower=-0.15 upper=3.14159 effort=500.0 velocity=200.0
- joint elbow_Z: limit lower=-3.14 upper=3.14 effort=500.0 velocity=200.0 -> lower=-0.15 upper=3.14 effort=500.0 velocity=200.0
- joint knee_Z: limit lower=-3.14 upper=3.14 effort=500.0 velocity=200.0 -> lower=-0.15 upper=2.80 effort=500.0 velocity=200.0
- joint lumbar_Z: limit lower=-3.14 upper=3.14 effort=500.0 velocity=200.0 -> lower=-2.0 upper=0.5 effort=500.0 velocity=200.0

Commit message: change from premanip thomas

File: urdf/human_5dof.urdf (robot description, URDF)
Before this commit: robot human_5dof, 8 links, 7 joints
Joints:
- joint elbow_Z: origin xyz=0.33566674458246937 0 0 rpy=0 -0 0 -> xyz=0.339 0 0 rpy=0 -0 0
- joint hand_fixed: origin xyz=0.23242554243018573 0 0 rpy=0 -0 0 -> xyz=0.2329 0 0 rpy=0 -0 0
- joint knee_Z: origin xyz=0.40155370945561 0 0 rpy=0 -0 0 -> xyz=0.4149 0 0 rpy=0 -0 0
- joint lumbar_Z: origin xyz=0.47648042433424215 0 0 rpy=0 -0 0 -> xyz=0.4766 0 0 rpy=0 -0 0
- joint shoulder_Z: origin xyz=0.4397691087116175 0 0 rpy=0 -0 0 -> xyz=0.4489 0 0 rpy=0 -0 0
- joint world_to_human: origin xyz=0.02373367081544142 0.005079786187961677 0.010846197486314102 rpy=1.572570285861921 0.15063584360293358 0.9840076914665431 -> xyz=0 0 0 rpy=1.57 0 0

Commit message: fix visuals

File: urdf/human_5dof.urdf (robot description, URDF)
Before this commit: robot human_5dof, 8 links, 7 joints
Links:
- link foot: geometry visual mesh filename=package://meshes/foot_mesh.STL scale=0.0060 0.0060 0.0060; visual mesh filename=package://meshes/foot_mesh.STL scale=0.0060 0.0060 0.0060
- link hand: geometry visual mesh filename=package://meshes/hand_mesh.STL scale=0.0060 0.0060 0.0060; visual mesh filename=package://meshes/hand_mesh.STL scale=0.0060 0.0060 0.0060
- link lowerarm: geometry visual mesh filename=package://meshes/elbow_mesh.STL scale=0.0055 0.0055 0.0055; visual mesh filename=package://meshes/elbow_mesh.STL scale=0.0055 0.0055 0.0055
- link lowerleg: geometry visual mesh filename=package://meshes/lowerleg_mesh.STL scale=0.0063 0.0065 0.007; visual mesh filename=package://meshes/lowerleg_mesh.STL scale=0.0063 0.0065 0.007
- link trunk: geometry visual mesh filename=package://meshes/abdomen_mesh.STL scale=0.0055 0.0055 0.0055; visual mesh filename=package://meshes/head_mesh.STL scale=0.0055 0.0055 0.0055
- link upperarm: geometry visual mesh filename=package://meshes/shoulder_mesh.STL scale=0.0055 0.0055 0.0055; visual mesh filename=package://meshes/shoulder_mesh.STL scale=0.0055 0.0055 0.0055
- link upperleg: geometry visual mesh filename=package://meshes/knee_mesh.STL scale=0.006 0.006 0.006; visual mesh filename=package://meshes/knee_mesh.STL scale=0.006 0.006 0.006
Joints:
- joint elbow_Z: origin xyz=0.361 0.0 0.0 rpy=0 -0 0 -> xyz=0.3465 0.0 0.0 rpy=0 -0 0
- joint hand_fixed: origin xyz=0.2666 0.0 0.0 rpy=0 -0 0 -> xyz=0.2732 0.0 0.0 rpy=0 -0 0
- joint knee_Z: origin xyz=0.428 0.0 0.0 rpy=0 -0 0 -> xyz=0.4571 0.0 0.0 rpy=0 -0 0
- joint lumbar_Z: origin xyz=0.5972 0.0 0.0 rpy=0 -0 0 -> xyz=0.6092 0.0 0.0 rpy=0 -0 0
- joint shoulder_Z: limit lower=-3.14 upper=1.54 effort=500.0 velocity=200.0 -> lower=-3.14 upper=3.14 effort=500.0 velocity=200.0; origin xyz=0.4706 0.0 0.0 rpy=0 -0 0 -> xyz=0.4811 0.0 0.0 rpy=0 -0 0

Commit message: sauvegarde du seum

File: urdf/human_5dof.urdf (robot description, URDF)
Before this commit: robot human_5dof, 8 links, 7 joints
Joints:
- joint elbow_Z: limit lower=-3.14159 upper=3.14159 effort=500.0 velocity=200.0 -> lower=-0.10 upper=2.96706 effort=500.0 velocity=200.0; origin xyz=0.3478 0.0 0.0 rpy=0 -0 0 -> xyz=0.3628 0.0 0.0 rpy=0 -0 0
- joint hand_fixed: origin xyz=0.2583 0.0 0.0 rpy=0 -0 0 -> xyz=0.2523 0.0 0.0 rpy=0 -0 0
- joint knee_Z: limit lower=-3.14159 upper=3.14159 effort=500.0 velocity=200.0 -> lower=-0.10 upper=3.14159 effort=500.0 velocity=200.0; origin xyz=0.4206 0.0 0.0 rpy=0 -0 0 -> xyz=0.4312 0.0 0.0 rpy=0 -0 0
- joint lumbar_Z: origin xyz=0.6008 0.0 0.0 rpy=0 -0 0 -> xyz=0.5519 0.0 0.0 rpy=0 -0 0
- joint shoulder_Z: limit lower=-6 upper=6 effort=500.0 velocity=200.0 -> lower=-4.01 upper=1.5708 effort=500.0 velocity=200.0; origin xyz=0.4944 0.0 0.0 rpy=0 -0 0 -> xyz=0.478 0.0 0.0 rpy=0 -0 0
- joint world_to_human: origin xyz=0.0005849673073485828 -0.000619424224471643 0.002751950406975956 rpy=1.5457406002736422 -0.060306077436283134 0.7220667584225953 -> xyz=-0.0 -0.0 -0.0 rpy=1.5707 0 0.78539

Commit message: calib redone and it seems better

File: urdf/human_5dof.urdf (robot description, URDF)
Before this commit: robot human_5dof, 8 links, 7 joints
Joints:
- joint elbow_Z: origin xyz=0.3628 0.0 0.0 rpy=0 -0 0 -> xyz=0.3465 0.0 0.0 rpy=0 -0 0
- joint hand_fixed: origin xyz=0.2523 0.0 0.0 rpy=0 -0 0 -> xyz=0.2732 0.0 0.0 rpy=0 -0 0
- joint knee_Z: origin xyz=0.4312 0.0 0.0 rpy=0 -0 0 -> xyz=0.4571 0.0 0.0 rpy=0 -0 0
- joint lumbar_Z: origin xyz=0.5519 0.0 0.0 rpy=0 -0 0 -> xyz=0.6092 0.0 0.0 rpy=0 -0 0
- joint shoulder_Z: origin xyz=0.478 0.0 0.0 rpy=0 -0 0 -> xyz=0.4811 0.0 0.0 rpy=0 -0 0
- joint world_to_human: origin xyz=-0.0 -0.0 -0.0 rpy=1.5707 0 0.78539 -> xyz=0.0 0.0 0.0 rpy=1.57 0.0 0.0

Commit message: new seztup

File: urdf/human_5dof.urdf (robot description, URDF)
Before this commit: robot human_5dof, 8 links, 7 joints
Joints:
- joint elbow_Z: origin xyz=0.3465 0.0 0.0 rpy=0 -0 0 -> xyz=0.3603 0.0 0.0 rpy=0 -0 0
- joint hand_fixed: origin xyz=0.2732 0.0 0.0 rpy=0 -0 0 -> xyz=0.2538 0.0 0.0 rpy=0 -0 0
- joint knee_Z: origin xyz=0.4571 0.0 0.0 rpy=0 -0 0 -> xyz=0.4492 0.0 0.0 rpy=0 -0 0
- joint lumbar_Z: origin xyz=0.6092 0.0 0.0 rpy=0 -0 0 -> xyz=0.5695 0.0 0.0 rpy=0 -0 0
- joint shoulder_Z: origin xyz=0.4811 0.0 0.0 rpy=0 -0 0 -> xyz=0.464 0.0 0.0 rpy=0 -0 0

Commit message: new setup calibration

File: urdf/human_5dof.urdf (robot description, URDF)
Before this commit: robot human_5dof, 8 links, 7 joints
Joints:
- joint elbow_Z: origin xyz=0.3603 0.0 0.0 rpy=0 -0 0 -> xyz=0.3285 0.0 0.0 rpy=0 -0 0
- joint hand_fixed: origin xyz=0.2538 0.0 0.0 rpy=0 -0 0 -> xyz=0.2327 0.0 0.0 rpy=0 -0 0
- joint knee_Z: origin xyz=0.4492 0.0 0.0 rpy=0 -0 0 -> xyz=0.368 0.0 0.0 rpy=0 -0 0
- joint lumbar_Z: origin xyz=0.5695 0.0 0.0 rpy=0 -0 0 -> xyz=0.4818 0.0 0.0 rpy=0 -0 0
- joint shoulder_Z: origin xyz=0.464 0.0 0.0 rpy=0 -0 0 -> xyz=0.4367 0.0 0.0 rpy=0 -0 0

Commit message: switching to qp for ik planar

File: urdf/human_5dof.urdf (robot description, URDF)
Before this commit: robot human_5dof, 8 links, 7 joints
Joints:
- joint elbow_Z: origin xyz=0.3285 0.0 0.0 rpy=0 -0 0 -> xyz=0.3052 0.0 0.0 rpy=0 -0 0
- joint hand_fixed: origin xyz=0.2327 0.0 0.0 rpy=0 -0 0 -> xyz=0.2173 0.0 0.0 rpy=0 -0 0
- joint knee_Z: origin xyz=0.368 0.0 0.0 rpy=0 -0 0 -> xyz=0.3751 0.0 0.0 rpy=0 -0 0
- joint lumbar_Z: origin xyz=0.4818 0.0 0.0 rpy=0 -0 0 -> xyz=0.4661 0.0 0.0 rpy=0 -0 0
- joint shoulder_Z: origin xyz=0.4367 0.0 0.0 rpy=0 -0 0 -> xyz=0.4305 0.0 0.0 rpy=0 -0 0
