Commit message: change the urdf to match the one from xacro and from the rest

File: urdf/5dof_mpc_base.urdf.xacro (robot description, xacro)
@@ -1,6 +1,21 @@
 <?xml version="1.0" encoding="utf-8"?>
-<robot xmlns:xacro="http://wiki.ros.org/xacro" name="human_5dof">
+<robot name = "human_5dof" xmlns:xacro="http://wiki.ros.org/xacro">
+<!-- Load the YAML files for calibration -->
+<xacro:property name="anthropometry_yaml_file" value="$(find rt-cosmik)/config/human_params/human_anthropometry.yaml"/>
+<xacro:property name="human_segment_lengths" value="${xacro.load_yaml(anthropometry_yaml_file)}"/>
+<xacro:property name="world_to_human_yaml_file" value="$(find rt-cosmik)/config/human_params/c1_human_color_test_test.yaml"/>
+<xacro:property name="human_base" value="${xacro.load_yaml(world_to_human_yaml_file)}"/>
+<!-- Properties -->
+<xacro:property name="translation" value="${human_base['translation_vector']['data']}" />
+<xacro:property name="rotation" value="${human_base['rotation_rpy']['data']}" />
+<xacro:property name="elbow_length" value="${human_segment_lengths['Elbow']}" />
+<xacro:property name="hip_length" value="${human_segment_lengths['Hip']}" />
+<xacro:property name="knee_length" value="${human_segment_lengths['Knee']}" />
+<xacro:property name="shoulder_length" value="${human_segment_lengths['Shoulder']}" />
+<xacro:property name="wrist_length" value="${human_segment_lengths['Wrist']}" />
+  <link name="world" />
   <joint name="world_to_human" type="fixed">
-    <origin rpy="1.57 -0 1.57" xyz="0.7 -1.25 0."/>
+    <origin xyz="${translation[0]} ${translation[1]} ${translation[2]}"
+            rpy="${rotation[0]} ${rotation[1]} ${rotation[2]}" />
     <axis xyz="0 0 1"/>
     <parent link="world"/>
@@ -14,24 +29,21 @@
     <inertial>
       <mass value="0.9" />
-      <origin xyz="0.068 -0.027 0.005" rpy="0 0 0" />
-      <inertia ixx="0.000815" ixy="0.000477" ixz="-0.00018" iyy="0.00386" iyz="0.0"
-        izz="0.003654" />
-    </inertial>
-    <visual>
-      <origin xyz="-0.05 0 0" rpy="0 1.57 0" />
-      <geometry>
-        <mesh filename="package://rt-cosmik/meshes/foot_mesh.STL"
-          scale="0.0060 0.0060 0.0060" />
-      </geometry>
-      <material name="body_color">
-        <texture />
-        <color rgba="0 1 1 0.5" />
-      </material>
-    </visual>
-    <visual>
-      <origin xyz="-0.05 0 0.15" rpy="0 1.57 0" />
-      <geometry>
-        <mesh filename="package://rt-cosmik/meshes/foot_mesh.STL"
-          scale="0.0060 0.0060 0.0060" />
+      <origin rpy="0 0 0" xyz="0.068 -0.027 0.005" />
+      <inertia ixx="0.000815" ixy="0.000477" ixz="-0.00018" iyy="0.00386" iyz="0.0" izz="0.003654" />
+    </inertial>
+    <visual>
+      <origin rpy="0 0 0" xyz="-0 0 0.1" />
+      <geometry>
+        <mesh filename="package://meshes/foot_mesh.STL" scale="0.0060 0.0060 0.0060" />
+      </geometry>
+      <material name="body_color">
+        <texture />
+        <color rgba="0 1 1 0.5" />
+      </material>
+    </visual>
+    <visual>
+      <origin rpy="0 0 0" xyz="0 0.0 -0.1" />
+      <geometry>
+        <mesh filename="package://meshes/foot_mesh.STL" scale="0.0060 0.0060 0.0060" />
       </geometry>
       <material name="body_color">
@@ -62,26 +74,21 @@
     <inertial>
       <mass value="3.6" />
-      <origin xyz="0.171 0.02 0.003" rpy="0 0 0" />
-      <inertia ixx="0.049314" ixy="-0.001006" ixz="-0.000252" iyy="0.00629" iyz="0.001573"
-        izz="0.049314" />
-    </inertial>
-    <visual>
-      <origin xyz="-0.0 0.06 0.0" rpy="1.57 1.57 0" />
-      <geometry>
-        <mesh
-          filename="package://rt-cosmik/meshes/lowerleg_mesh.STL"
-          scale="0.0063 0.0065 0.007" />
-      </geometry>
-      <material name="body_color">
-        <texture />
-        <color rgba="0 1 1 0.5" />
-      </material>
-    </visual>
-    <visual>
-      <origin xyz="-0.0 0.06 0.155" rpy="1.57 1.57 0" />
-      <geometry>
-        <mesh
-          filename="package://rt-cosmik/meshes/lowerleg_mesh.STL"
-          scale="0.0063 0.0065 0.007" />
+      <origin rpy="0 -0 0" xyz="0.171 0.02 0.003" />
+      <inertia ixx="0.049314" ixy="-0.001006" ixz="-0.000252" iyy="0.00629" iyz="0.001573" izz="0.049314" />
+    </inertial>
+    <visual>
+      <origin rpy="0 0 -1.57" xyz="0.45 0.0 0.1" />
+      <geometry>
+        <mesh filename="package://meshes/lowerleg_mesh.STL" scale="0.0063 0.0065 0.007" />
+      </geometry>
+      <material name="body_color">
+        <texture />
+        <color rgba="0 1 1 0.5" />
+      </material>
+    </visual>
+    <visual>
+      <origin rpy="0 0 -1.57" xyz="0.45 0.0 -0.1" />
+      <geometry>
+        <mesh filename="package://meshes/lowerleg_mesh.STL" scale="0.0063 0.0065 0.007" />
       </geometry>
       <material name="body_color">
@@ -92,5 +99,5 @@
   </link>
   <joint name="knee_Z" type="revolute">
-    <origin rpy="0 -0 0" xyz="0.38 0.0 0.0" />
+    <origin rpy="0 -0 0" xyz="${knee_length} 0.0 0.0"/>
     <axis xyz="0 0 1" />
     <parent link="lowerleg" />
@@ -112,48 +119,41 @@
     <inertial>
       <mass value="9.22" />
-      <origin xyz="0.179 0.017 0.014" rpy="0 0 0" />
-      <inertia ixx="0.134834" ixy="0.007856" ixz="-0.000641" iyy="0.036073" iyz="-0.007856"
-        izz="0.144293" />
-    </inertial>
-    <visual>
-      <origin xyz="-0.06 -0.05 -0.12" rpy="0.0 0 0" />
-      <geometry>
-        <mesh filename="package://rt-cosmik/meshes/knee_mesh.STL"
-          scale="0.006 0.006 0.006" />
-      </geometry>
-      <material name="body_color">
-        <texture />
-        <color rgba="0 1 1 0.5" />
-      </material>
-    </visual>
-    <visual>
-      <origin xyz="-0.06 -0.05 0.03" rpy="0.0 0 0" />
-      <geometry>
-        <mesh filename="package://rt-cosmik/meshes/knee_mesh.STL"
-          scale="0.006 0.006 0.006" />
-      </geometry>
-      <material name="body_color">
-        <texture />
-        <color rgba="0 1 1 0.5" />
-      </material>
-    </visual>
-    <visual>
-      <origin xyz="0.02 0.07 0" rpy="1.57 1.57 0" />
-      <geometry>
-        <mesh
-          filename="package://rt-cosmik/meshes/upperleg_mesh.STL"
-          scale="0.0063 0.0065 0.007" />
-      </geometry>
-      <material name="body_color">
-        <texture />
-        <color rgba="0 1 1 0.5" />
-      </material>
-    </visual>
-    <visual>
-      <origin xyz="0.02 0.07 0.155" rpy="1.57 1.57 0" />
-      <geometry>
-        <mesh
-          filename="package://rt-cosmik/meshes/upperleg_mesh.STL"
-          scale="0.0063 0.0065 0.007" />
+      <origin rpy="0 -0 0" xyz="0.179 0.017 0.014" />
+      <inertia ixx="0.134834" ixy="0.007856" ixz="-0.000641" iyy="0.036073" iyz="-0.007856" izz="0.144293" />
+    </inertial>
+    <visual>
+      <origin rpy="0.0 0 -1.57" xyz="0.05 0.0 0.1" />
+      <geometry>
+        <mesh filename="package://meshes/knee_mesh.STL" scale="0.006 0.006 0.006" />
+      </geometry>
+      <material name="body_color">
+        <texture />
+        <color rgba="0 1 1 0.5" />
+      </material>
+    </visual>
+    <visual>
+      <origin rpy="0.0 0 -1.57" xyz="0.05 0.0 -0.1" />
+      <geometry>
+        <mesh filename="package://meshes/knee_mesh.STL" scale="0.006 0.006 0.006" />
+      </geometry>
+      <material name="body_color">
+        <texture />
+        <color rgba="0 1 1 0.5" />
+      </material>
+    </visual>
+    <visual>
+      <origin rpy="0 0 -1.57" xyz="0.47 0.0 0.1" />
+      <geometry>
+        <mesh filename="package://meshes/upperleg_mesh.STL" scale="0.0063 0.0065 0.007" />
+      </geometry>
+      <material name="body_color">
+        <texture />
+        <color rgba="0 1 1 0.5" />
+      </material>
+    </visual>
+    <visual>
+      <origin rpy="0 0 -1.57" xyz="0.47 0.0 -0.1" />
+      <geometry>
+        <mesh filename="package://meshes/upperleg_mesh.STL" scale="0.0063 0.0065 0.007" />
       </geometry>
       <material name="body_color">
@@ -164,5 +164,5 @@
   </link>
   <joint name="lumbar_Z" type="revolute">
-    <origin rpy="0 -0 0" xyz="0.48 0.0 0.0" />
+    <origin rpy="0 -0 0" xyz="${hip_length} 0.0 0.0"/>
     <axis xyz="0 0 1" />
     <parent link="upperleg" />
@@ -184,37 +184,31 @@
     <inertial>
       <mass value="35.47" />
-      <origin xyz="0.116 0.007 -0.001" rpy="0 0 0" />
-      <inertia ixx="2.592457" ixy="7.005900e-02" ixz="-3.523000e-04" iyy="2.448720e-01"
-        iyz="-4.236600e-03" izz="2.594914" />
-    </inertial>
-    <visual>
-      <origin xyz="-0.043 0.105 0.125" rpy="1.57 1.57 0" />
-      <geometry>
-        <mesh
-          filename="package://rt-cosmik/meshes/pelvis_mesh.STL"
-          scale="0.006 0.0055 0.0055" />
-      </geometry>
-      <material name="body_color">
-        <texture />
-        <color rgba="0 1 1 0.5" />
-      </material>
-    </visual>
-    <visual>
-      <origin xyz="0.10 -0.085 -0.085" rpy="0 0 0" />
-      <geometry>
-        <mesh
-          filename="package://rt-cosmik/meshes/abdomen_mesh.STL"
-          scale="0.0055 0.0055 0.0055" />
-      </geometry>
-      <material name="body_color">
-        <texture />
-        <color rgba="0 1 1 0.5" />
-      </material>
-    </visual>
-    <visual>
-      <origin xyz="0.22 0.13 0.125" rpy="1.57 1.57 0" />
-      <geometry>
-        <mesh filename="package://rt-cosmik/meshes/torso_mesh.STL"
-          scale="0.0065 0.0065 0.0065" />
+      <origin rpy="0 -0 0" xyz="0.116 0.007 -0.001" />
+      <inertia ixx="2.592457" ixy="7.005900e-02" ixz="-3.523000e-04" iyy="2.448720e-01" iyz="-4.236600e-03" izz="2.594914" />
+    </inertial>
+    <visual>
+      <origin rpy="0 0 -1.57" xyz="0.05 0.0 0.0" />
+      <geometry>
+        <mesh filename="package://meshes/pelvis_mesh.STL" scale="0.006 0.0055 0.0055" />
+      </geometry>
+      <material name="body_color">
+        <texture />
+        <color rgba="0 1 1 0.5" />
+      </material>
+    </visual>
+    <visual>
+      <origin rpy="0 -0 -1.57" xyz="0.06 0.0 0.0" />
+      <geometry>
+        <mesh filename="package://meshes/abdomen_mesh.STL" scale="0.0055 0.0055 0.0055" />
+      </geometry>
+      <material name="body_color">
+        <texture />
+        <color rgba="0 1 1 0.5" />
+      </material>
+    </visual>
+    <visual>
+      <origin rpy="0 0 -1.57" xyz="0.0 0.0 0.0" />
+      <geometry>
+        <mesh filename="package://meshes/torso_mesh.STL" scale="0.0065 0.0065 0.0065" />
       </geometry>
       <material name="body_color">
@@ -224,8 +218,7 @@
     </visual>
     <visual>
-      <origin xyz="0.57 0.085 0.085" rpy="1.57 1.57 0" />
-      <geometry>
-        <mesh filename="package://rt-cosmik/meshes/head_mesh.STL"
-          scale="0.0055 0.0055 0.0055" />
+      <origin rpy="0 0 -1.57" xyz="0.5 0.0 0.0" />
+      <geometry>
+        <mesh filename="package://meshes/head_mesh.STL" scale="0.0055 0.0055 0.0055" />
       </geometry>
       <material name="body_color">
@@ -235,8 +228,7 @@
     </visual>
     <visual>
-      <origin xyz="0.51 -0.05 -0.05" rpy="0 0.0 0" />
-      <geometry>
-        <mesh filename="package://rt-cosmik/meshes/neck_mesh.STL"
-          scale="0.005 0.005 0.005" />
+      <origin rpy="0 0.0 0" xyz="0.5 -0.0 0.0" />
+      <geometry>
+        <mesh filename="package://meshes/neck_mesh.STL" scale="0.005 0.005 0.005" />
       </geometry>
       <material name="body_color">
@@ -247,5 +239,5 @@
   </link>
   <joint name="shoulder_Z" type="revolute">
-    <origin rpy="0 -0 0" xyz="0.45 0.0 0.0" />
+    <origin rpy="0 -0 0" xyz="${shoulder_length} 0.0 0.0"/>
     <axis xyz="0 0 1" />
     <parent link="trunk" />
@@ -267,47 +259,38 @@
     <inertial>
       <mass value="1.8" />
-      <origin xyz="0.118 -0.004 -0.007" rpy="0 0 0" />
-      <inertia ixx="0.011874" ixy="0.000445" ixz="0.000309" iyy="0.002422" iyz="4.9e-05"
-        izz="0.012652" />
-    </inertial>
-    <visual>
-      <origin xyz="-0.15 -0.05 0.12" rpy="0 0 0" />
-      <geometry>
-        <mesh
-          filename="package://rt-cosmik/meshes/shoulder_mesh.STL"
-          scale="0.0055 0.0055 0.0055" />
-      </geometry>
-      <material name="body_color">
-        <texture />
-        <color rgba="0 1 1 0.5" />
-      </material>
-    </visual>
-    <visual>
-      <origin xyz="-0.02 -0.065 -0.355" rpy="1.57 -1.57 3.14" />
-      <geometry>
-        <mesh
-          filename="package://rt-cosmik/meshes/upperarm_mesh.STL"
-          scale="0.0063 0.0060 0.007" />
+      <origin rpy="0 -0 0" xyz="0.118 -0.004 -0.007" />
+      <inertia ixx="0.011874" ixy="0.000445" ixz="0.000309" iyy="0.002422" iyz="4.9e-05" izz="0.012652" />
+    </inertial>
+    <visual>
+      <origin rpy="0 0 1.57" xyz="0.0 0.0 0.15" />
+      <geometry>
+        <mesh filename="package://meshes/shoulder_mesh.STL" scale="0.0055 0.0055 0.0055" />
+      </geometry>
+      <material name="body_color">
+        <texture />
+        <color rgba="0 1 1 0.5" />
+      </material>
+    </visual>
+    <visual>
+      <origin rpy="0 0 1.57" xyz="0.0 0.0 0.15" />
+      <geometry>
+        <mesh filename="package://meshes/upperarm_mesh.STL" scale="0.0063 0.0060 0.007" />
       </geometry>
       <material name="body_color" />
     </visual>
     <visual>
-      <origin xyz="-0.15 -0.05 -0.225" rpy="0 0 0" />
-      <geometry>
-        <mesh
-          filename="package://rt-cosmik/meshes/shoulder_mesh.STL"
-          scale="0.0055 0.0055 0.0055" />
-      </geometry>
-      <material name="body_color">
-        <texture />
-        <color rgba="0 1 1 0.5" />
-      </material>
-    </visual>
-    <visual>
-      <origin xyz="-0.02 -0.065 -0.01" rpy="1.57 -1.57 3.14" />
-      <geometry>
-        <mesh
-          filename="package://rt-cosmik/meshes/upperarm_mesh.STL"
-          scale="0.0063 0.0060 0.007" />
+      <origin rpy="0 0 1.57" xyz="0.0 0.0 -0.15" />
+      <geometry>
+        <mesh filename="package://meshes/shoulder_mesh.STL" scale="0.0055 0.0055 0.0055" />
+      </geometry>
+      <material name="body_color">
+        <texture />
+        <color rgba="0 1 1 0.5" />
+      </material>
+    </visual>
+    <visual>
+      <origin rpy="0 0 1.57" xyz="0.0 0.0 -0.15" />
+      <geometry>
+        <mesh filename="package://meshes/upperarm_mesh.STL" scale="0.0063 0.0060 0.007" />
       </geometry>
       <material name="body_color" />
@@ -315,5 +298,5 @@
   </link>
   <joint name="elbow_Z" type="revolute">
-    <origin rpy="0 -0 0" xyz="0.29 0.0 0.0" />
+    <origin rpy="0 -0 0" xyz="${elbow_length} 0.0 0.0"/>
     <axis xyz="0 0 1" />
     <parent link="upperarm" />
@@ -335,48 +318,41 @@
     <inertial>
       <mass value="1.28" />
-      <origin xyz="0.114 -0.003 0.004" rpy="0 0 0" />
-      <inertia ixx="0.007479" ixy="8.6e-05" ixz="3.8e-05" iyy="0.001154" iyz="-0.000611"
-        izz="0.006954" />
-    </inertial>
-    <visual>
-      <origin xyz="-0.165 -0.035 -0.21" rpy="0 0 0" />
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
File: urdf/human_5dof.urdf (robot description, URDF)
Before this commit: robot human_5dof, 8 links, 7 joints
Links:
- link foot: geometry visual mesh filename=package://rt-cosmik/meshes/foot_mesh.STL scale=0.0060 0.0060 0.0060; visual mesh filename=package://rt-cosmik/meshes/foot_mesh.STL scale=0.0060 0.0060 0.0060
- link hand: geometry visual mesh filename=package://rt-cosmik/meshes/hand_mesh.STL scale=0.0060 0.0060 0.0060; visual mesh filename=package://rt-cosmik/meshes/hand_mesh.STL scale=0.0060 0.0060 0.0060
- link lowerarm: geometry visual mesh filename=package://rt-cosmik/meshes/elbow_mesh.STL scale=0.0055 0.0055 0.0055; visual mesh filename=package://rt-cosmik/meshes/elbow_mesh.STL scale=0.0055 0.0055 0.0055
- link lowerleg: geometry visual mesh filename=package://rt-cosmik/meshes/lowerleg_mesh.STL scale=0.0063 0.0065 0.007; visual mesh filename=package://rt-cosmik/meshes/lowerleg_mesh.STL scale=0.0063 0.0065 0.007
- link trunk: geometry visual mesh filename=package://rt-cosmik/meshes/abdomen_mesh.STL scale=0.0055 0.0055 0.0055; visual mesh filename=package://rt-cosmik/meshes/head_mesh.STL scale=0.0055 0.0055 0.0055
- link upperarm: geometry visual mesh filename=package://rt-cosmik/meshes/shoulder_mesh.STL scale=0.0055 0.0055 0.0055; visual mesh filename=package://rt-cosmik/meshes/shoulder_mesh.STL scale=0.0055 0.0055 0.0055
- link upperleg: geometry visual mesh filename=package://rt-cosmik/meshes/knee_mesh.STL scale=0.006 0.006 0.006; visual mesh filename=package://rt-cosmik/meshes/knee_mesh.STL scale=0.006 0.006 0.006
Joints:
- joint ankle_Z: limit lower=-0.15 upper=3.14159 effort=500.0 velocity=200.0 -> lower=-0.785398 upper=3.14159 effort=500.0 velocity=200.0
- joint elbow_Z: limit lower=-0.15 upper=3.14 effort=500.0 velocity=200.0 -> lower=0 upper=2.74889 effort=500.0 velocity=200.0; origin xyz=0.339 0 0 rpy=0 -0 0 -> xyz=0.361 0.0 0.0 rpy=0 -0 0
- joint hand_fixed: origin xyz=0.2329 0 0 rpy=0 -0 0 -> xyz=0.2666 0.0 0.0 rpy=0 -0 0
- joint knee_Z: limit lower=-0.15 upper=2.80 effort=500.0 velocity=200.0 -> lower=-2.74889 upper=2.74889 effort=500.0 velocity=200.0; origin xyz=0.4149 0 0 rpy=0 -0 0 -> xyz=0.428 0.0 0.0 rpy=0 -0 0
- joint lumbar_Z: limit lower=-2.0 upper=0.5 effort=500.0 velocity=200.0 -> lower=-3.14 upper=0 effort=500.0 velocity=200.0; origin xyz=0.4766 0 0 rpy=0 -0 0 -> xyz=0.5972 0.0 0.0 rpy=0 -0 0
- joint shoulder_Z: limit lower=-3.14 upper=3.14 effort=500.0 velocity=200.0 -> lower=-3.14 upper=1.54 effort=500.0 velocity=200.0; origin xyz=0.4489 0 0 rpy=0 -0 0 -> xyz=0.4706 0.0 0.0 rpy=0 -0 0
- joint world_to_human: origin xyz=0 0 0 rpy=1.57 0 0 -> xyz=0.0005849673073485828 -0.000619424224471643 0.002751950406975956 rpy=1.5457406002736422 -0.060306077436283134 0.7220667584225953

Commit message: change shoulder bounds

File: urdf/5dof_mpc_base.urdf.xacro (robot description, xacro)
@@ -243,5 +243,5 @@
     <parent link="trunk" />
     <child link="upperarm" />
-    <limit effort="500.0" velocity="200.0" lower="-3.14" upper="1.54" />
+    <limit effort="500.0" velocity="200.0" lower="-3.14" upper="3.14" />
   </joint>
   <!-- TRANSMITION DEFINITION -->

Commit message: change bounds model

File: urdf/5dof_mpc_base.urdf.xacro (robot description, xacro)
@@ -58,5 +58,5 @@
     <parent link="foot" />
     <child link="lowerleg" />
-    <limit effort="500.0" velocity="200.0" lower="-0.785398" upper="3.14159" />
+    <limit effort="500.0" velocity="200.0" lower="-3.14159" upper="3.14159" />
   </joint>
   <!-- TRANSMITION DEFINITION -->
@@ -103,5 +103,5 @@
     <parent link="lowerleg" />
     <child link="upperleg" />
-    <limit effort="500.0" velocity="200.0" lower="-2.74889" upper="2.74889" />
+    <limit effort="500.0" velocity="200.0" lower="-0.10" upper="3.14159" />
   </joint>
   <!-- TRANSMITION DEFINITION -->
@@ -168,5 +168,5 @@
     <parent link="upperleg" />
     <child link="trunk" />
-    <limit effort="500.0" velocity="200.0" lower="-3.14" upper="0" />
+    <limit effort="500.0" velocity="200.0" lower="-3.14" upper="3.14159" />
   </joint>
   <!-- TRANSMITION DEFINITION -->
@@ -243,5 +243,5 @@
     <parent link="trunk" />
     <child link="upperarm" />
-    <limit effort="500.0" velocity="200.0" lower="-3.14" upper="3.14" />
+    <limit effort="500.0" velocity="200.0" lower="-6" upper="6" />
   </joint>
   <!-- TRANSMITION DEFINITION -->
@@ -302,5 +302,5 @@
     <parent link="upperarm" />
     <child link="lowerarm" />
-    <limit effort="500.0" velocity="200.0" lower="0" upper="2.74889" />
+    <limit effort="500.0" velocity="200.0" lower="-3.14159" upper="3.14159" />
   </joint>
   <!-- TRANSMITION DEFINITION -->

File: urdf/human_5dof.urdf (robot description, URDF)
Before this commit: robot human_5dof, 8 links, 7 joints
Joints:
- joint ankle_Z: limit lower=-0.785398 upper=3.14159 effort=500.0 velocity=200.0 -> lower=-3.14159 upper=3.14159 effort=500.0 velocity=200.0
- joint elbow_Z: limit lower=0 upper=2.74889 effort=500.0 velocity=200.0 -> lower=-3.14159 upper=3.14159 effort=500.0 velocity=200.0; origin xyz=0.3465 0.0 0.0 rpy=0 -0 0 -> xyz=0.3478 0.0 0.0 rpy=0 -0 0
- joint hand_fixed: origin xyz=0.2732 0.0 0.0 rpy=0 -0 0 -> xyz=0.2583 0.0 0.0 rpy=0 -0 0
- joint knee_Z: limit lower=-2.74889 upper=2.74889 effort=500.0 velocity=200.0 -> lower=-3.14159 upper=3.14159 effort=500.0 velocity=200.0; origin xyz=0.4571 0.0 0.0 rpy=0 -0 0 -> xyz=0.4206 0.0 0.0 rpy=0 -0 0
- joint lumbar_Z: limit lower=-3.14 upper=0 effort=500.0 velocity=200.0 -> lower=-3.14 upper=3.14159 effort=500.0 velocity=200.0; origin xyz=0.6092 0.0 0.0 rpy=0 -0 0 -> xyz=0.6008 0.0 0.0 rpy=0 -0 0
- joint shoulder_Z: limit lower=-3.14 upper=3.14 effort=500.0 velocity=200.0 -> lower=-6 upper=6 effort=500.0 velocity=200.0; origin xyz=0.4811 0.0 0.0 rpy=0 -0 0 -> xyz=0.4944 0.0 0.0 rpy=0 -0 0

Commit message: change bounds

File: urdf/5dof_mpc_base.urdf.xacro (robot description, xacro)
@@ -243,5 +243,5 @@
     <parent link="trunk" />
     <child link="upperarm" />
-    <limit effort="500.0" velocity="200.0" lower="-6" upper="6" />
+    <limit effort="500.0" velocity="200.0" lower="-4.01" upper="1.5708" />
   </joint>
   <!-- TRANSMITION DEFINITION -->
@@ -302,5 +302,5 @@
     <parent link="upperarm" />
     <child link="lowerarm" />
-    <limit effort="500.0" velocity="200.0" lower="-3.14159" upper="3.14159" />
+    <limit effort="500.0" velocity="200.0" lower="-0.10" upper="2,96706" />
   </joint>
   <!-- TRANSMITION DEFINITION -->

Commit message: fixes

File: urdf/5dof_mpc_base.urdf.xacro (robot description, xacro)
@@ -302,5 +302,5 @@
     <parent link="upperarm" />
     <child link="lowerarm" />
-    <limit effort="500.0" velocity="200.0" lower="-0.10" upper="2,96706" />
+    <limit effort="500.0" velocity="200.0" lower="-0.10" upper="2.96706" />
   </joint>
   <!-- TRANSMITION DEFINITION -->

Commit message: change in hands ori

File: urdf/5dof_mpc_base.urdf.xacro (robot description, xacro)
@@ -376,5 +376,5 @@
     </inertial>
     <visual>
-      <origin rpy="0 0 1.57" xyz="0.035 0.0 0.15" />
+      <origin rpy="0 1.57 1.57" xyz="0.035 0.0 0.15" />
       <geometry>
         <mesh filename="package://meshes/hand_mesh.STL" scale="0.0060 0.0060 0.0060" />
@@ -386,5 +386,5 @@
     </visual>
     <visual>
-      <origin rpy="0 0 1.57" xyz="0.035 0.0 -0.15" />
+      <origin rpy="0 -1.57 1.57" xyz="0.035 0.0 -0.15" />
       <geometry>
         <mesh filename="package://meshes/hand_mesh.STL" scale="0.0060 0.0060 0.0060" />
