Commit message: test ik and full pipeline should be tested on gpu

File: urdf/2dof_human_arm_polishing.urdf (robot description, URDF)
Before this commit: robot human_2dof_planar_model, 4 links, 3 joints
Joints:
- removed joint elbow_Z
- removed joint shoulder_Z
- added joint elbow: type revolute, parent upperarm, child lowerarm, origin xyz=0.262 0.0 0.0 rpy=0 -0 0, axis 0 -1 0, limit lower=0 upper=2.74889 effort=0 velocity=0
- added joint shoulder: type revolute, parent trunk, child upperarm, origin xyz=0.0 0.0 0.0 rpy=0 0 0, axis 0 -1 0, limit lower=-1.5708 upper=1.5708 effort=0 velocity=0
