Commit message: fix paths meshes

File: urdf/human.urdf (robot description, URDF)
Before this commit: robot human_wb, 24 links, 23 joints
Links:
- link footL: geometry visual mesh filename=package://rt-cosmik/meshes/foot_mesh.STL scale=0.0060 0.0060 0.0060
- link footR: geometry visual mesh filename=package://rt-cosmik/meshes/foot_mesh.STL scale=0.0060 0.0060 0.0060
- link lowerarmL: geometry visual mesh filename=package://rt-cosmik/meshes/lowerarm_mesh.STL scale=0.0060 0.0060 0.0060
- link lowerarmR: geometry visual mesh filename=package://rt-cosmik/meshes/lowerarm_mesh.STL scale=0.0060 0.0060 0.0060
- link lowerarm_z: geometry visual mesh filename=package://rt-cosmik/meshes/elbow_mesh.STL scale=0.0055 0.0055 0.0055
- link lowerarm_z_L: geometry visual mesh filename=package://rt-cosmik/meshes/elbow_mesh.STL scale=0.0055 0.0055 0.0055
- link pelvis: geometry visual mesh filename=package://rt-cosmik/meshes/pelvis_mesh.STL scale=0.006 0.0055 0.0055
- link shankL: geometry visual mesh filename=package://rt-cosmik/meshes/lowerleg_mesh.STL scale=0.0063 0.0065 0.007
- link shankR: geometry visual mesh filename=package://rt-cosmik/meshes/lowerleg_mesh.STL scale=0.0063 0.0065 0.007
- link thighL: geometry visual mesh filename=package://rt-cosmik/meshes/upperleg_mesh.STL scale=0.0063 0.0065 0.007
- link thighR: geometry visual mesh filename=package://rt-cosmik/meshes/upperleg_mesh.STL scale=0.0063 0.0065 0.007
- link thigh_x: geometry visual mesh filename=package://rt-cosmik/meshes/knee_mesh.STL scale=0.006 0.006 0.006
- link thigh_x_L: geometry visual mesh filename=package://rt-cosmik/meshes/knee_mesh.STL scale=0.006 0.006 0.006
- link torso: geometry visual mesh filename=package://rt-cosmik/meshes/abdomen_mesh.STL scale=0.0055 0.0055 0.0055; visual mesh filename=package://rt-cosmik/meshes/torso_mesh.STL scale=0.0065 0.0065 0.0065
- link upperarmL: geometry visual mesh filename=package://rt-cosmik/meshes/upperarm_mesh.STL scale=0.0063 0.0060 0.007
- link upperarmR: geometry visual mesh filename=package://rt-cosmik/meshes/upperarm_mesh.STL scale=0.0063 0.0060 0.007
- link upperarm_z_L: geometry visual mesh filename=package://rt-cosmik/meshes/shoulder_mesh.STL scale=0.0055 0.0055 0.0055
- link upperarm_z_R: geometry visual mesh filename=package://rt-cosmik/meshes/shoulder_mesh.STL scale=0.0055 0.0055 0.0055

File: urdf/human.urdf.xacro (robot description, xacro)
@@ -21,5 +21,5 @@
 	        <origin xyz="-0.08 -0.13 0.125" rpy="0 1.57 0" />
             <geometry>
-		        <mesh filename="package://rt_cosmik/meshes/pelvis_mesh.STL" scale="0.006 0.0055 0.0055"/>
+		        <mesh filename="package://rt-cosmik/meshes/pelvis_mesh.STL" scale="0.006 0.0055 0.0055"/>
             </geometry>
             <material name="body_color">
@@ -53,5 +53,5 @@
             <origin xyz="-0.05 0.05 -0.085" rpy="0 -0 0" />
             <geometry>
-		        <mesh filename="package://rt_cosmik/meshes/abdomen_mesh.STL" scale="0.0055 0.0055 0.0055"/>
+		        <mesh filename="package://rt-cosmik/meshes/abdomen_mesh.STL" scale="0.0055 0.0055 0.0055"/>
                 <!--<box size="0.15 0.161217 0.198658" />-->
             </geometry>
@@ -65,5 +65,5 @@
             <geometry>
 		        <!--<box size="0.15 0.356643 0.329994" />-->
-		        <mesh filename="package://rt_cosmik/meshes/torso_mesh.STL" scale="0.0065 0.0065 0.0065"/>
+		        <mesh filename="package://rt-cosmik/meshes/torso_mesh.STL" scale="0.0065 0.0065 0.0065"/>
             </geometry>
             <material name="body_color">
@@ -84,5 +84,5 @@
 	        <origin xyz="-0.15 -0.04 -0.05" rpy="0 0 0" />
             <geometry>
-		        <mesh filename="package://rt_cosmik/meshes/shoulder_mesh.STL" scale="0.0055 0.0055 0.0055"/>
+		        <mesh filename="package://rt-cosmik/meshes/shoulder_mesh.STL" scale="0.0055 0.0055 0.0055"/>
             </geometry>
             <material name="body_color">
@@ -116,5 +116,5 @@
             <origin xyz="-0.065 -0.27 0.18" rpy="0.0 1.57 0" />
             <geometry>
-                <mesh filename="package://rt_cosmik/meshes/upperarm_mesh.STL" scale="0.0063 0.0060 0.007"/>
+                <mesh filename="package://rt-cosmik/meshes/upperarm_mesh.STL" scale="0.0063 0.0060 0.007"/>
             </geometry>
             <material name="body_color">
@@ -135,5 +135,5 @@
 	        <origin xyz="-0.15 -0.04 -0.035" rpy="0 0 0" />
             <geometry>
-		        <mesh filename="package://rt_cosmik/meshes/elbow_mesh.STL" scale="0.0055 0.0055 0.0055"/>
+		        <mesh filename="package://rt-cosmik/meshes/elbow_mesh.STL" scale="0.0055 0.0055 0.0055"/>
             </geometry>
             <material name="body_color">
@@ -159,5 +159,5 @@
             <origin xyz="0.052 -0.26 -0.17" rpy="0.0 -1.57 0" />
             <geometry>
-                <mesh filename="package://rt_cosmik/meshes/lowerarm_mesh.STL" scale="0.0060 0.0060 0.0060"/>
+                <mesh filename="package://rt-cosmik/meshes/lowerarm_mesh.STL" scale="0.0060 0.0060 0.0060"/>
             </geometry>
             <material name="body_color">
@@ -178,5 +178,5 @@
 	        <origin xyz="-0.16 -0.045 -0.045" rpy="0 0 0" />
             <geometry>
-		        <mesh filename="package://rt_cosmik/meshes/shoulder_mesh.STL" scale="0.0055 0.0055 0.0055"/>
+		        <mesh filename="package://rt-cosmik/meshes/shoulder_mesh.STL" scale="0.0055 0.0055 0.0055"/>
             </geometry>
             <material name="body_color">
@@ -210,5 +210,5 @@
             <origin xyz="-0.065 -0.27 0.18" rpy="0.0 1.57 0" />
             <geometry>
-                <mesh filename="package://rt_cosmik/meshes/upperarm_mesh.STL" scale="0.0063 0.0060 0.007"/>
+                <mesh filename="package://rt-cosmik/meshes/upperarm_mesh.STL" scale="0.0063 0.0060 0.007"/>
             </geometry>
             <material name="body_color"/>
@@ -226,5 +226,5 @@
 	        <origin xyz="-0.15 -0.04 -0.035" rpy="0 0 0" />
             <geometry>
-		        <mesh filename="package://rt_cosmik/meshes/elbow_mesh.STL" scale="0.0055 0.0055 0.0055"/>
+		        <mesh filename="package://rt-cosmik/meshes/elbow_mesh.STL" scale="0.0055 0.0055 0.0055"/>
             </geometry>
             <material name="body_color">
@@ -250,5 +250,5 @@
             <origin xyz="0.052 -0.26 -0.17" rpy="0.0 -1.57 0" />
             <geometry>
-                <mesh filename="package://rt_cosmik/meshes/lowerarm_mesh.STL" scale="0.0060 0.0060 0.0060"/>
+                <mesh filename="package://rt-cosmik/meshes/lowerarm_mesh.STL" scale="0.0060 0.0060 0.0060"/>
             </geometry>
             <material name="body_color">
@@ -277,5 +277,5 @@
             <origin xyz="-0.04 -0.48 0.07" rpy="0.0 1.57 0" />
             <geometry>
-                <mesh filename="package://rt_cosmik/meshes/knee_mesh.STL" scale="0.006 0.006 0.006"/>
+                <mesh filename="package://rt-cosmik/meshes/knee_mesh.STL" scale="0.006 0.006 0.006"/>
             </geometry>
             <material name="body_color">
@@ -301,5 +301,5 @@
             <origin xyz="-0.1 -0.42 0.07" rpy="0.0 1.57 0" />
             <geometry>
-                <mesh filename="package://rt_cosmik/meshes/upperleg_mesh.STL" scale="0.0063 0.0065 0.007"/>
+                <mesh filename="package://rt-cosmik/meshes/upperleg_mesh.STL" scale="0.0063 0.0065 0.007"/>
             </geometry>
             <material name="body_color">
@@ -325,5 +325,5 @@
             <origin xyz="-0.06 -0.43 0.07" rpy="0.0 1.57 0" />
             <geometry>
-                <mesh filename="package://rt_cosmik/meshes/lowerleg_mesh.STL" scale="0.0063 0.0065 0.007"/>
+                <mesh filename="package://rt-cosmik/meshes/lowerleg_mesh.STL" scale="0.0063 0.0065 0.007"/>
             </geometry>
             <material name="body_color">
@@ -349,5 +349,5 @@
             <origin xyz="-0.05 -0.055 0.065" rpy="0 1.57 0" />
             <geometry>
-		        <mesh filename="package://rt_cosmik/meshes/foot_mesh.STL" scale="0.0060 0.0060 0.0060"/>
+		        <mesh filename="package://rt-cosmik/meshes/foot_mesh.STL" scale="0.0060 0.0060 0.0060"/>
                 <!--<box size="0.03 0.085239 0.06" />-->
             </geometry>
@@ -377,5 +377,5 @@
             <origin xyz="-0.04 -0.48 0.080" rpy="0.0 1.57 0" />
             <geometry>
-                <mesh filename="package://rt_cosmik/meshes/knee_mesh.STL" scale="0.006 0.006 0.006"/>
+                <mesh filename="package://rt-cosmik/meshes/knee_mesh.STL" scale="0.006 0.006 0.006"/>
             </geometry>
             <material name="body_color">
@@ -401,5 +401,5 @@
             <origin xyz="-0.1 -0.42 0.085" rpy="0.0 1.57 0" />
             <geometry>
-                <mesh filename="package://rt_cosmik/meshes/upperleg_mesh.STL" scale="0.0063 0.0065 0.007"/>
+                <mesh filename="package://rt-cosmik/meshes/upperleg_mesh.STL" scale="0.0063 0.0065 0.007"/>
             </geometry>
             <material name="body_color">
@@ -425,5 +425,5 @@
             <origin xyz="-0.06 -0.43 0.08" rpy="0.0 1.57 0" />
             <geometry>
-                <mesh filename="package://rt_cosmik/meshes/lowerleg_mesh.STL" scale="0.0063 0.0065 0.007"/>
+                <mesh filename="package://rt-cosmik/meshes/lowerleg_mesh.STL" scale="0.0063 0.0065 0.007"/>
             </geometry>
             <material name="body_color">
@@ -449,5 +449,5 @@
             <origin xyz="-0.05 -0.055 0.075" rpy="0 1.57 0" />
             <geometry>
-		        <mesh filename="package://rt_cosmik/meshes/foot_mesh.STL" scale="0.0060 0.0060 0.0060"/>
+		        <mesh filename="package://rt-cosmik/meshes/foot_mesh.STL" scale="0.0060 0.0060 0.0060"/>
                 <!--<box size="0.03 0.085239 0.06" />-->
             </geometry>

File: urdf/human_5dof.urdf (robot description, URDF)
Before this commit: robot human_5dof, 8 links, 7 joints
Links:
- link foot: geometry visual mesh filename=package://rt-cosmik/meshes/foot_mesh.STL scale=0.0060 0.0060 0.0060; visual mesh filename=package://rt-cosmik/meshes/foot_mesh.STL scale=0.0060 0.0060 0.0060
- link hand: geometry visual mesh filename=package://rt-cosmik/meshes/hand_mesh.STL scale=0.0060 0.0060 0.0060; visual mesh filename=package://rt-cosmik/meshes/hand_mesh.STL scale=0.0060 0.0060 0.0060
- link lowerarm: geometry visual mesh filename=package://rt-cosmik/meshes/elbow_mesh.STL scale=0.0055 0.0055 0.0055; visual mesh filename=package://rt-cosmik/meshes/elbow_mesh.STL scale=0.0055 0.0055 0.0055
- link lowerleg: geometry visual mesh filename=package://rt-cosmik/meshes/lowerleg_mesh.STL scale=0.0063 0.0065 0.007; visual mesh filename=package://rt-cosmik/meshes/lowerleg_mesh.STL scale=0.0063 0.0065 0.007
- link trunk: geometry visual mesh filename=package://rt-cosmik/meshes/abdomen_mesh.STL scale=0.0055 0.0055 0.0055; visual mesh filename=package://rt-cosmik/meshes/head_mesh.STL scale=0.0055 0.0055 0.0055
- link upperarm: geometry visual mesh filename=package://rt-cosmik/meshes/shoulder_mesh.STL scale=0.0055 0.0055 0.0055; visual mesh filename=package://rt-cosmik/meshes/shoulder_mesh.STL scale=0.0055 0.0055 0.0055
- link upperleg: geometry visual mesh filename=package://rt-cosmik/meshes/knee_mesh.STL scale=0.006 0.006 0.006; visual mesh filename=package://rt-cosmik/meshes/knee_mesh.STL scale=0.006 0.006 0.006

Commit message: Features/new visual

File: urdf/human.urdf (robot description, URDF)
Before this commit: robot human_wb, 24 links, 23 joints
Links:
- link footL: geometry visual mesh filename=package://meshes/foot_mesh.STL scale=0.0060 0.0060 0.0060
- link footR: geometry visual mesh filename=package://meshes/foot_mesh.STL scale=0.0060 0.0060 0.0060
- link lowerarmL: geometry visual mesh filename=package://meshes/lowerarm_mesh.STL scale=0.0060 0.0060 0.0060
- link lowerarmR: geometry visual mesh filename=package://meshes/lowerarm_mesh.STL scale=0.0060 0.0060 0.0060
- link lowerarm_z: geometry visual mesh filename=package://meshes/elbow_mesh.STL scale=0.0055 0.0055 0.0055
- link lowerarm_z_L: geometry visual mesh filename=package://meshes/elbow_mesh.STL scale=0.0055 0.0055 0.0055
- link pelvis: geometry visual mesh filename=package://meshes/pelvis_mesh.STL scale=0.006 0.0055 0.0055
- link shankL: geometry visual mesh filename=package://meshes/knee_mesh.STL scale=0.006 0.006 0.006; visual mesh filename=package://meshes/lowerleg_mesh.STL scale=0.0063 0.0065 0.007
- link shankR: geometry visual mesh filename=package://meshes/knee_mesh.STL scale=0.006 0.006 0.006; visual mesh filename=package://meshes/lowerleg_mesh.STL scale=0.0063 0.0065 0.007
- link thighL: geometry visual mesh filename=package://meshes/upperleg_mesh.STL scale=0.0063 0.0065 0.007
- link thighR: geometry visual mesh filename=package://meshes/upperleg_mesh.STL scale=0.0063 0.0065 0.007
- link thigh_x: geometry 
- link thigh_x_L: geometry 
- link torso: geometry visual mesh filename=package://meshes/abdomen_mesh.STL scale=0.0055 0.0055 0.0055; visual mesh filename=package://meshes/torso_mesh.STL scale=0.0065 0.0065 0.0065
- link upperarmL: geometry visual mesh filename=package://meshes/upperarm_mesh.STL scale=0.0063 0.0060 0.007
- link upperarmR: geometry visual mesh filename=package://meshes/upperarm_mesh.STL scale=0.0063 0.0060 0.007
- link upperarm_z_L: geometry visual mesh filename=package://meshes/shoulder_mesh.STL scale=0.0055 0.0055 0.0055
- link upperarm_z_R: geometry visual mesh filename=package://meshes/shoulder_mesh.STL scale=0.0055 0.0055 0.0055

File: urdf/human.urdf.xacro (robot description, xacro)
@@ -19,5 +19,5 @@
         </inertial>
         <visual>
-	        <origin xyz="-0.08 -0.13 0.125" rpy="0 1.57 0" />
+	        <origin xyz="0. 0. 0." rpy="0 0 0" />
             <geometry>
 		        <mesh filename="package://rt-cosmik/meshes/pelvis_mesh.STL" scale="0.006 0.0055 0.0055"/>
@@ -51,5 +51,5 @@
         </inertial>
         <visual>
-            <origin xyz="-0.05 0.05 -0.085" rpy="0 -0 0" />
+            <origin xyz="0. 0. 0." rpy="0 -0 0" />
             <geometry>
 		        <mesh filename="package://rt-cosmik/meshes/abdomen_mesh.STL" scale="0.0055 0.0055 0.0055"/>
@@ -62,5 +62,5 @@
         </visual>
         <visual>
-	    <origin xyz="-0.115 0.17 0.125" rpy="0 1.57 0" />
+	    <origin xyz="0. 0. 0." rpy="0 0 0" />
             <geometry>
 		        <!--<box size="0.15 0.356643 0.329994" />-->
@@ -82,5 +82,5 @@
     <link name="upperarm_z_R">
         <visual>
-	        <origin xyz="-0.15 -0.04 -0.05" rpy="0 0 0" />
+	        <origin xyz="0. 0. 0." rpy="0 0 0" />
             <geometry>
 		        <mesh filename="package://rt-cosmik/meshes/shoulder_mesh.STL" scale="0.0055 0.0055 0.0055"/>
@@ -114,5 +114,5 @@
         </inertial>
         <visual>
-            <origin xyz="-0.065 -0.27 0.18" rpy="0.0 1.57 0" />
+            <origin xyz="0.0 0. 0." rpy="0.0 0 0" />
             <geometry>
                 <mesh filename="package://rt-cosmik/meshes/upperarm_mesh.STL" scale="0.0063 0.0060 0.007"/>
@@ -133,5 +133,5 @@
     <link name="lowerarm_z">
         <visual>
-	        <origin xyz="-0.15 -0.04 -0.035" rpy="0 0 0" />
+	        <origin xyz="0. 0. 0." rpy="0 0 0" />
             <geometry>
 		        <mesh filename="package://rt-cosmik/meshes/elbow_mesh.STL" scale="0.0055 0.0055 0.0055"/>
@@ -157,5 +157,5 @@
         </inertial>
         <visual>
-            <origin xyz="0.052 -0.26 -0.17" rpy="0.0 -1.57 0" />
+            <origin xyz="0. 0. 0." rpy="0.0 0 0" />
             <geometry>
                 <mesh filename="package://rt-cosmik/meshes/lowerarm_mesh.STL" scale="0.0060 0.0060 0.0060"/>
@@ -176,5 +176,5 @@
     <link name="upperarm_z_L">
 	    <visual>
-	        <origin xyz="-0.16 -0.045 -0.045" rpy="0 0 0" />
+	        <origin xyz="0. 0. 0." rpy="0 0 0" />
             <geometry>
 		        <mesh filename="package://rt-cosmik/meshes/shoulder_mesh.STL" scale="0.0055 0.0055 0.0055"/>
@@ -208,5 +208,5 @@
         </inertial>
         <visual>
-            <origin xyz="-0.065 -0.27 0.18" rpy="0.0 1.57 0" />
+            <origin xyz="0. 0. 0." rpy="0.0 0 0" />
             <geometry>
                 <mesh filename="package://rt-cosmik/meshes/upperarm_mesh.STL" scale="0.0063 0.0060 0.007"/>
@@ -224,5 +224,5 @@
     <link name="lowerarm_z_L">
 	    <visual>
-	        <origin xyz="-0.15 -0.04 -0.035" rpy="0 0 0" />
+	        <origin xyz="0. 0. 0." rpy="0 0 0" />
             <geometry>
 		        <mesh filename="package://rt-cosmik/meshes/elbow_mesh.STL" scale="0.0055 0.0055 0.0055"/>
@@ -248,5 +248,5 @@
         </inertial>
         <visual>
-            <origin xyz="0.052 -0.26 -0.17" rpy="0.0 -1.57 0" />
+            <origin xyz="0. 0. 0." rpy="0.0 0 0" />
             <geometry>
                 <mesh filename="package://rt-cosmik/meshes/lowerarm_mesh.STL" scale="0.0060 0.0060 0.0060"/>
@@ -274,14 +274,4 @@
     </joint>
     <link name="thigh_x">
-        <visual>
-            <origin xyz="-0.04 -0.48 0.07" rpy="0.0 1.57 0" />
-            <geometry>
-                <mesh filename="package://rt-cosmik/meshes/knee_mesh.STL" scale="0.006 0.006 0.006"/>
-            </geometry>
-            <material name="body_color">
-                <texture />
-                <color rgba="0 1 1 0.5" />
-            </material>
-        </visual>
     </link>
     <joint name="right_hip_Y" type="revolute">
@@ -299,5 +289,5 @@
         </inertial>
         <visual>
-            <origin xyz="-0.1 -0.42 0.07" rpy="0.0 1.57 0" />
+            <origin xyz="0. 0. 0." rpy="0.0 0 0" />
             <geometry>
                 <mesh filename="package://rt-cosmik/meshes/upperleg_mesh.STL" scale="0.0063 0.0065 0.007"/>
@@ -323,7 +313,17 @@
         </inertial>
         <visual>
-            <origin xyz="-0.06 -0.43 0.07" rpy="0.0 1.57 0" />
+            <origin xyz="0. 0. 0." rpy="0.0 0 0" />
             <geometry>
                 <mesh filename="package://rt-cosmik/meshes/lowerleg_mesh.STL" scale="0.0063 0.0065 0.007"/>
+            </geometry>
+            <material name="body_color">
+                <texture />
+                <color rgba="0 1 1 0.5" />
+            </material>
+        </visual>
+                <visual>
+            <origin xyz="0. 0. 0." rpy="0.0 0 0" />
+            <geometry>
+                <mesh filename="package://rt-cosmik/meshes/knee_mesh.STL" scale="0.006 0.006 0.006"/>
             </geometry>
             <material name="body_color">
@@ -347,5 +347,5 @@
         </inertial>
         <visual>
-            <origin xyz="-0.05 -0.055 0.065" rpy="0 1.57 0" />
+            <origin xyz="0. 0. 0." rpy="0 0 0" />
             <geometry>
 		        <mesh filename="package://rt-cosmik/meshes/foot_mesh.STL" scale="0.0060 0.0060 0.0060"/>
@@ -374,14 +374,4 @@
     </joint>
     <link name="thigh_x_L">
-	    <visual>
-            <origin xyz="-0.04 -0.48 0.080" rpy="0.0 1.57 0" />
-            <geometry>
-                <mesh filename="package://rt-cosmik/meshes/knee_mesh.STL" scale="0.006 0.006 0.006"/>
-            </geometry>
-            <material name="body_color">
-                <texture />
-                <color rgba="0 1 1 0.5" />
-            </material>
-        </visual>
     </link>
     <joint name="left_hip_Y" type="revolute">
@@ -399,5 +389,5 @@
         </inertial>
         <visual>
-            <origin xyz="-0.1 -0.42 0.085" rpy="0.0 1.57 0" />
+            <origin xyz="0. -0. 0." rpy="0.0 0 0" />
             <geometry>
                 <mesh filename="package://rt-cosmik/meshes/upperleg_mesh.STL" scale="0.0063 0.0065 0.007"/>
@@ -423,5 +413,5 @@
         </inertial>
         <visual>
-            <origin xyz="-0.06 -0.43 0.08" rpy="0.0 1.57 0" />
+            <origin xyz="0. 0. 0." rpy="0.0 0 0" />
             <geometry>
                 <mesh filename="package://rt-cosmik/meshes/lowerleg_mesh.STL" scale="0.0063 0.0065 0.007"/>
@@ -432,4 +422,14 @@
             </material>
 	    </visual>
+        	    <visual>
+            <origin xyz="0. 0. 0." rpy="0.0 0 0" />
+            <geometry>
+                <mesh filename="package://rt-cosmik/meshes/knee_mesh.STL" scale="0.006 0.006 0.006"/>
+            </geometry>
+            <material name="body_color">
+                <texture />
+                <color rgba="0 1 1 0.5" />
+            </material>
+        </visual>
     </link>
     <joint name="left_ankle_Z" type="revolute">
@@ -447,5 +447,5 @@
         </inertial>
         <visual>
-            <origin xyz="-0.05 -0.055 0.075" rpy="0 1.57 0" />
+            <origin xyz="0. 0. 0." rpy="0 0 0" />
             <geometry>
 		        <mesh filename="package://rt-cosmik/meshes/foot_mesh.STL" scale="0.0060 0.0060 0.0060"/>

File: urdf/human_5dof.urdf (robot description, URDF)
Before this commit: robot human_5dof, 8 links, 7 joints
Links:
- link foot: geometry visual mesh filename=package://meshes/foot_mesh.STL scale=0.0060 0.0060 0.0060; visual mesh filename=package://meshes/foot_mesh.STL scale=0.0060 0.0060 0.0060
- link hand: geometry visual mesh filename=package://meshes/hand_mesh.STL scale=0.0060 0.0060 0.0060; visual mesh filename=package://meshes/hand_mesh.STL scale=0.0060 0.0060 0.0060
- link lowerarm: geometry visual mesh filename=package://meshes/elbow_mesh.STL scale=0.0055 0.0055 0.0055; visual mesh filename=package://meshes/elbow_mesh.STL scale=0.0055 0.0055 0.0055
- link lowerleg: geometry visual mesh filename=package://meshes/lowerleg_mesh.STL scale=0.0063 0.0065 0.007; visual mesh filename=package://meshes/lowerleg_mesh.STL scale=0.0063 0.0065 0.007
- link trunk: geometry visual mesh filename=package://meshes/abdomen_mesh.STL scale=0.0055 0.0055 0.0055; visual mesh filename=package://meshes/head_mesh.STL scale=0.0055 0.0055 0.0055
- link upperarm: geometry visual mesh filename=package://meshes/shoulder_mesh.STL scale=0.0055 0.0055 0.0055; visual mesh filename=package://meshes/shoulder_mesh.STL scale=0.0055 0.0055 0.0055
- link upperleg: geometry visual mesh filename=package://meshes/knee_mesh.STL scale=0.006 0.006 0.006; visual mesh filename=package://meshes/knee_mesh.STL scale=0.006 0.006 0.006
