Commit message: adaptation of full model

File: urdf/human.urdf (robot description, URDF)
Before this commit: robot human_wb, 24 links, 23 joints
Links:
- removed link footL
- removed link footR
- removed link lowerarmL
- removed link lowerarmR
- removed link lowerarm_z
- removed link lowerarm_z_L
- removed link pelvis
- removed link shankL
- removed link shankR
- removed link thighL
- removed link thighR
- removed link thigh_x
- removed link thigh_x_L
- removed link thigh_z
- removed link thigh_z_L
- removed link torso
- removed link torso_z
- removed link upperarmL
- removed link upperarmR
- removed link upperarm_x_L
- removed link upperarm_x_R
- removed link upperarm_z_L
- removed link upperarm_z_R
- removed link world
- added link left_clavicle, mass 0.15600
- added link left_foot, mass 1.13208; visual mesh filename=meshes/foot_mesh.STL scale=0.0060 0.0060 0.0060
- added link left_foot_virtual
- added link left_hand, mass 0.56604; visual mesh filename=meshes/hand_mesh.STL scale=0.0060 0.0060 0.0060
- added link left_hand_virtual
- added link left_lowerarm, mass 1.60378; visual mesh filename=meshes/lowerarm_mesh.STL scale=0.0060 0.0060 0.0060
- added link left_lowerarm_virtual; visual mesh filename=meshes/elbow_mesh.STL scale=0.0055 0.0055 0.0055
- added link left_lowerleg, mass 4.52832; visual mesh filename=meshes/lowerleg_mesh.STL scale=0.0063 0.0065 0.007
- added link left_upperarm, mass 2.26416; visual mesh filename=meshes/upperarm_mesh.STL scale=0.0063 0.0060 0.007
- added link left_upperarm_virtual; visual mesh filename=meshes/shoulder_mesh.STL scale=0.0055 0.0055 0.0055
- added link left_upperarm_virtual_2
- added link left_upperleg, mass 11.6038; visual mesh filename=meshes/upperleg_mesh.STL scale=0.0063 0.0065 0.007
- added link left_upperleg_virtual
- added link left_upperleg_virtual_2; visual mesh filename=meshes/knee_mesh.STL scale=0.006 0.006 0.006
- added link middle_abdomen, mass 2.73586; visual mesh filename=meshes/abdomen_mesh.STL scale=0.0055 0.0055 0.0055
- added link middle_abdomen_virtual
- added link middle_head, mass 6.32078; visual mesh filename=meshes/head_mesh.STL scale=0.0055 0.0055 0.0055
- added link middle_head_virtual; visual mesh filename=meshes/neck_mesh.STL scale=0.005 0.005 0.005
- added link middle_head_virtual_2
- added link middle_pelvis, mass 13.3963; visual mesh filename=meshes/pelvis_mesh.STL scale=0.006 0.0055 0.0055
- added link middle_thorax, mass 28.6794; visual mesh filename=meshes/torso_mesh.STL scale=0.0065 0.0065 0.0065
- added link middle_thorax_virtual
- added link middle_thorax_virtual_2
- added link right_clavicle, mass 0.15600
- added link right_foot, mass 1.13208; visual mesh filename=meshes/foot_mesh.STL scale=0.0060 0.0060 0.0060
- added link right_foot_virtual
- added link right_hand, mass 0.56604; visual mesh filename=meshes/hand_mesh.STL scale=0.0060 0.0060 0.0060
- added link right_hand_virtual
- added link right_lowerarm, mass 1.60378; visual mesh filename=meshes/lowerarm_mesh.STL scale=0.0060 0.0060 0.0060
- added link right_lowerarm_virtual; visual mesh filename=meshes/elbow_mesh.STL scale=0.0055 0.0055 0.0055
- added link right_lowerleg, mass 4.52832; visual mesh filename=meshes/lowerleg_mesh.STL scale=0.0063 0.0065 0.007
- added link right_upperarm, mass 2.26416; visual mesh filename=meshes/upperarm_mesh.STL scale=0.0063 0.0060 0.007
- added link right_upperarm_virtual; visual mesh filename=meshes/shoulder_mesh.STL scale=0.0055 0.0055 0.0055
- added link right_upperarm_virtual_2
- added link right_upperleg, mass 11.6038; visual mesh filename=meshes/upperleg_mesh.STL scale=0.0063 0.0065 0.007
- added link right_upperleg_virtual
- added link right_upperleg_virtual_2; visual mesh filename=meshes/knee_mesh.STL scale=0.006 0.006 0.006
Joints:
- removed joint left_knee_Z
- removed joint middle_lumbar_Y
- removed joint right_knee_Z
- removed joint world_to_human
- added joint left_ankle_X: type revolute, parent left_foot_virtual, child left_foot, origin xyz=0 0 0 rpy=0 -0 0, axis -1 0 0, limit lower=-0.523598333 upper=0.785398 effort=20 velocity=0
- added joint left_clavicle_joint_X: type revolute, parent middle_thorax, child left_clavicle, origin xyz=0 0.330225 0 rpy=0 -0 0, axis 1 0 0, limit lower=-1.0472 upper=0.314159 effort=0 velocity=0
- added joint left_knee: type revolute, parent left_upperleg, child left_lowerleg, origin xyz=0 -0.427 0 rpy=0 -0 0, axis 0 0 -1, limit lower=0 upper=3.14159 effort=168 velocity=0
- added joint left_wrist_X: type revolute, parent left_hand_virtual, child left_hand, origin xyz=0 0 0 rpy=0 -0 0, axis -1 0 0, limit lower=-0.785398 upper=0.785398 effort=0 velocity=0
- added joint left_wrist_Z: type revolute, parent left_lowerarm, child left_hand_virtual, origin xyz=0 -0.27965 0 rpy=0 -0 0, axis 0 0 1, limit lower=-1.5708 upper=1.5708 effort=185 velocity=0
- added joint middle_cervical_X: type revolute, parent middle_head_virtual, child middle_head_virtual_2, origin xyz=0 0 0 rpy=0 -0 0, axis 1 0 0, limit lower=-1.5708 upper=1.5708 effort=0 velocity=0
- added joint middle_cervical_Y: type revolute, parent middle_head_virtual_2, child middle_head, origin xyz=0 0 0 rpy=0 -0 0, axis 0 1 0, limit lower=-1.5708 upper=1.5708 effort=0 velocity=0
- added joint middle_cervical_Z: type revolute, parent middle_thorax, child middle_head_virtual, origin xyz=0 0.330225 0 rpy=0 -0 0, axis 0 0 -1, limit lower=-1.5708 upper=1.5708 effort=0 velocity=0
- added joint middle_lumbar_X: type revolute, parent middle_abdomen_virtual, child middle_abdomen, origin xyz=0 0 0 rpy=0 -0 0, axis 1 0 0, limit lower=-0.785398 upper=0.785398 effort=159 velocity=0
- added joint middle_thoracic_X: type revolute, parent middle_thorax_virtual, child middle_thorax_virtual_2, origin xyz=0 0 0 rpy=0 -0 0, axis 1 0 0, limit lower=-1.0472 upper=1.0472 effort=159 velocity=0
- added joint middle_thoracic_Y: type revolute, parent middle_thorax_virtual_2, child middle_thorax, origin xyz=0 0 0 rpy=0 -0 0, axis 0 1 0, limit lower=-1.0472 upper=1.0472 effort=159 velocity=0
- added joint middle_thoracic_Z: type revolute, parent middle_abdomen, child middle_thorax_virtual, origin xyz=0 0.149275 0 rpy=0 -0 0, axis 0 0 -1, limit lower=-1.0472 upper=0.392699 effort=159 velocity=0
- added joint right_ankle_X: type revolute, parent right_foot_virtual, child right_foot, origin xyz=0 0 0 rpy=0 -0 0, axis 1 0 0, limit lower=-0.523598333 upper=0.785398 effort=20 velocity=0
- added joint right_clavicle_joint_X: type revolute, parent middle_thorax, child right_clavicle, origin xyz=0 0.330225 0 rpy=0 -0 0, axis -1 0 0, limit lower=-0.392699 upper=1.0472 effort=0 velocity=0
- added joint right_knee: type revolute, parent right_upperleg, child right_lowerleg, origin xyz=0 -0.427 0 rpy=0 -0 0, axis 0 0 -1, limit lower=0 upper=3.14159 effort=168 velocity=0
- added joint right_wrist_X: type revolute, parent right_hand_virtual, child right_hand, origin xyz=0 0 0 rpy=0 -0 0, axis 1 0 0, limit lower=-0.785398 upper=0.785398 effort=0 velocity=0
- added joint right_wrist_Z: type revolute, parent right_lowerarm, child right_hand_virtual, origin xyz=0 -0.27965 0 rpy=0 -0 0, axis 0 0 1, limit lower=-1.5708 upper=1.5708 effort=185 velocity=0
- joint left_ankle_Z: child footL -> left_foot_virtual; limit lower=-0.392699 upper=1.0472 effort=0 velocity=0 -> lower=-1.570795 upper=0.7853975 effort=126 velocity=0; parent shankL -> left_lowerleg
- joint left_elbow_Y: child lowerarmL -> left_lowerarm; limit lower=-1.5708 upper=1.5708 effort=0 velocity=0 -> lower=-3.14159 upper=0.2 effort=15 velocity=0; parent lowerarm_z_L -> left_lowerarm_virtual
- joint left_elbow_Z: child lowerarm_z_L -> left_lowerarm_virtual; limit lower=0 upper=2.74889 effort=0 velocity=0 -> lower=0 upper=2.617991667 effort=77 velocity=0; parent upperarmL -> left_upperarm
- joint left_hip_X: child thigh_x_L -> left_upperleg_virtual_2; limit lower=-0.392699 upper=1.5708 effort=0 velocity=0 -> lower=-1.047196667 upper=1.570795 effort=190 velocity=0; parent thigh_z_L -> left_upperleg_virtual
- joint left_hip_Y: child thighL -> left_upperleg; limit lower=-1.5708 upper=1.5708 effort=0 velocity=0 -> lower=-1.047196667 upper=1.570795 effort=60 velocity=0; parent thigh_x_L -> left_upperleg_virtual_2
- joint left_hip_Z: child thigh_z_L -> left_upperleg_virtual; limit lower=-0.785398 upper=3.14159 effort=0 velocity=0 -> lower=-1.047196667 upper=3.14159 effort=190 velocity=0; parent pelvis -> middle_pelvis
- joint left_shoulder_X: child upperarm_x_L -> left_upperarm_virtual_2; limit lower=-3.14159 upper=1.0472 effort=0 velocity=0 -> lower=-1.0472 upper=3.14159 effort=71 velocity=0; parent upperarm_z_L -> left_upperarm_virtual
- joint left_shoulder_Y: child upperarmL -> left_upperarm; parent upperarm_x_L -> left_upperarm_virtual_2
- joint left_shoulder_Z: child upperarm_z_L -> left_upperarm_virtual; limit lower=-2.0944 upper=0.392699 effort=0 velocity=0 -> lower=-3.14159 upper=3.14159 effort=92 velocity=0; origin xyz=0.00805 0.4067 -0.2037 rpy=0 -0 0 -> xyz=0.00805 -0.0728 -0.2037 rpy=0 -0 0; parent torso -> left_clavicle
- joint middle_lumbar_Z: axis 0 0 1 -> 0 0 -1; child torso_z -> middle_abdomen_virtual; limit lower=-3.14159 upper=0.785398 effort=0 velocity=0 -> lower=-3.14159 upper=0.785398 effort=243 velocity=0; parent pelvis -> middle_pelvis
- joint right_ankle_Z: child footR -> right_foot_virtual; limit lower=-1.0472 upper=0.392699 effort=0 velocity=0 -> lower=-1.570795 upper=0.7853975 effort=126 velocity=0; parent shankR -> right_lowerleg
- joint right_elbow_Y: child lowerarmR -> right_lowerarm; limit lower=-1.5708 upper=1.5708 effort=0 velocity=0 -> lower=-0.2 upper=3.14159 effort=15 velocity=0; parent lowerarm_z -> right_lowerarm_virtual
- joint right_elbow_Z: child lowerarm_z -> right_lowerarm_virtual; limit lower=0 upper=2.74889 effort=0 velocity=0 -> lower=0 upper=2.617991667 effort=77 velocity=0; parent upperarmR -> right_upperarm
- joint right_hip_X: child thigh_x -> right_upperleg_virtual_2; limit lower=-0.392699 upper=1.5708 effort=0 velocity=0 -> lower=-1.570795 upper=1.047196667 effort=190 velocity=0; parent thigh_z -> right_upperleg_virtual
- joint right_hip_Y: child thighR -> right_upperleg; limit lower=-1.5708 upper=1.5708 effort=0 velocity=0 -> lower=-1.570795 upper=1.047196667 effort=190 velocity=0; parent thigh_x -> right_upperleg_virtual_2
- joint right_hip_Z: child thigh_z -> right_upperleg_virtual; limit lower=-0.785398 upper=3.14159 effort=0 velocity=0 -> lower=-1.047196667 upper=3.14159 effort=190 velocity=0; parent pelvis -> middle_pelvis
- joint right_shoulder_X: axis 1 0 0 -> -1 0 0; child upperarm_x_R -> right_upperarm_virtual_2; limit lower=-3.14159 upper=1.0472 effort=0 velocity=0 -> lower=-1.0472 upper=3.14159 effort=71 velocity=0; parent upperarm_z_R -> right_upperarm_virtual
- joint right_shoulder_Y: axis 0 1 0 -> 0 -1 0; child upperarmR -> right_upperarm; parent upperarm_x_R -> right_upperarm_virtual_2
- joint right_shoulder_Z: child upperarm_z_R -> right_upperarm_virtual; limit lower=-2.0944 upper=0.392699 effort=0 velocity=0 -> lower=-3.14159 upper=3.14159 effort=0 velocity=0; origin xyz=0.00805 0.4067 0.2037 rpy=0 -0 0 -> xyz=0.00805 -0.0728 0.2037 rpy=0 -0 0; parent torso -> right_clavicle

Commit message: launch swika,ipopt on all data

File: urdf/human.urdf (robot description, URDF)
Before this commit: robot human_36dof_ISB_model, 37 links, 36 joints
Links:
- link left_foot: mass 1.13208 -> 0.9; geometry visual mesh filename=meshes/foot_mesh.STL scale=0.0067 0.0067 0.0067
- link left_hand: mass 0.56604 -> 0.45; geometry visual mesh filename=meshes/hand_mesh.STL scale=0.0061 0.0061 0.0061
- link left_lowerarm: mass 1.60378 -> 1.28; geometry visual mesh filename=meshes/elbow_mesh.STL scale=0.0055 0.0055 0.0055; visual mesh filename=meshes/lowerarm_mesh.STL scale=0.0064 0.0064 0.0064
- link left_lowerarm_virtual: geometry 
- link left_lowerleg: mass 4.52832 -> 3.6; geometry visual mesh filename=meshes/knee_mesh.STL scale=0.0056 0.0056 0.0056; visual mesh filename=meshes/lowerleg_mesh.STL scale=0.0063 0.0066 0.007
- link left_upperarm: mass 2.26416 -> 1.8; geometry visual mesh filename=meshes/shoulder_mesh.STL scale=0.0039 0.0039 0.0039; visual mesh filename=meshes/upperarm_mesh.STL scale=0.0063 0.006 0.0069
- link left_upperarm_virtual: geometry 
- link left_upperleg: mass 11.6038 -> 9.22; geometry visual mesh filename=meshes/upperleg_mesh.STL scale=0.0062 0.0064 0.0069
- link left_upperleg_virtual_2: geometry 
- link middle_abdomen: mass 2.73586 -> 12.25; geometry visual mesh filename=meshes/abdomen_mesh.STL scale=0.0074 0.0074 0.0074
- link middle_head: mass 6.32078 -> 5.03; geometry visual mesh filename=meshes/head_mesh.STL scale=0.0056 0.0056 0.0056; visual mesh filename=meshes/neck_mesh.STL scale=0.005 0.005 0.005
- link middle_head_virtual: geometry 
- link middle_pelvis: mass 13.3963 -> 10.65; geometry visual mesh filename=meshes/pelvis_mesh.STL scale=0.0063 0.0058 0.0058
- link middle_thorax: mass 28.6794 -> 11.97; geometry visual mesh filename=meshes/torso_mesh.STL scale=0.007 0.007 0.007
- link right_foot: mass 1.13208 -> 0.9; geometry visual mesh filename=meshes/foot_mesh.STL scale=0.0067 0.0067 0.0067
- link right_hand: mass 0.56604 -> 0.45; geometry visual mesh filename=meshes/hand_mesh.STL scale=0.0061 0.0061 0.0061
- link right_lowerarm: mass 1.60378 -> 1.28; geometry visual mesh filename=meshes/elbow_mesh.STL scale=0.0055 0.0055 0.0055; visual mesh filename=meshes/lowerarm_mesh.STL scale=0.0064 0.0064 0.0064
- link right_lowerarm_virtual: geometry 
- link right_lowerleg: mass 4.52832 -> 3.6; geometry visual mesh filename=meshes/knee_mesh.STL scale=0.0056 0.0056 0.0056; visual mesh filename=meshes/lowerleg_mesh.STL scale=0.0063 0.0066 0.007
- link right_upperarm: mass 2.26416 -> 1.8; geometry visual mesh filename=meshes/shoulder_mesh.STL scale=0.0039 0.0039 0.0039; visual mesh filename=meshes/upperarm_mesh.STL scale=0.0063 0.006 0.0069
- link right_upperarm_virtual: geometry 
- link right_upperleg: mass 11.6038 -> 9.22; geometry visual mesh filename=meshes/upperleg_mesh.STL scale=0.0062 0.0064 0.0069
- link right_upperleg_virtual_2: geometry 
Joints:
- removed joint left_knee
- removed joint right_knee
- added joint left_knee_Z: type revolute, parent left_upperleg, child left_lowerleg, origin xyz=0. -0.439 0. rpy=0 -0 0, axis 0 0 -1, limit lower=0 upper=3.14159 effort=130 velocity=18.6
- added joint right_knee_Z: type revolute, parent right_upperleg, child right_lowerleg, origin xyz=0 -0.439 0 rpy=0 -0 0, axis 0 0 -1, limit lower=0 upper=3.14159 effort=130 velocity=18.6
- joint left_ankle_X: limit lower=-0.523598333 upper=0.785398 effort=20 velocity=0 -> lower=-0.523598333 upper=0.785398 effort=20 velocity=2.0
- joint left_ankle_Z: limit lower=-1.570795 upper=0.7853975 effort=126 velocity=0 -> lower=-1.570795 upper=0.7853975 effort=126 velocity=12.7; origin xyz=0 -0.42805 0 rpy=0 -0 0 -> xyz=0 -0.44 0 rpy=0 -0 0
- joint left_clavicle_joint_X: limit lower=-1.0472 upper=0.314159 effort=0 velocity=0 -> lower=-0.349066 upper=1.0472 effort=100 velocity=14.0; origin xyz=0 0.330225 0 rpy=0 -0 0 -> xyz=0 0.176 0 rpy=0 -0 0
- joint left_elbow_Y: axis 0 1 0 -> 0 -1 0; limit lower=-3.14159 upper=0.2 effort=15 velocity=0 -> lower=-0.349066 upper=3.14159 effort=15 velocity=6.0
- joint left_elbow_Z: limit lower=0 upper=2.617991667 effort=77 velocity=0 -> lower=0 upper=2.617991667 effort=77 velocity=19.9; origin xyz=0 -0.2737 0 rpy=0 -0 0 -> xyz=0 -0.276 0 rpy=0 -0 0
- joint left_hip_X: limit lower=-1.047196667 upper=1.570795 effort=190 velocity=0 -> lower=-1.047196667 upper=1.570795 effort=120 velocity=12.0
- joint left_hip_Y: axis 0 1 0 -> 0 -1 0; limit lower=-1.047196667 upper=1.570795 effort=60 velocity=0 -> lower=-1.570795 upper=1.047196667 effort=60 velocity=12.0
- joint left_hip_Z: limit lower=-1.047196667 upper=3.14159 effort=190 velocity=0 -> lower=-1.047196667 upper=3.14159 effort=185 velocity=12.0; origin xyz=0.053375 -0.0749 -0.079975 rpy=0 -0 0 -> xyz=0.023 -0.1 -0.082 rpy=0 -0 0
- joint left_shoulder_X: limit lower=-1.0472 upper=3.14159 effort=71 velocity=0 -> lower=-1.0472 upper=3.14159 effort=71 velocity=6.0
- joint left_shoulder_Y: axis 0 1 0 -> 0 -1 0; limit lower=-1.5708 upper=3.14159 effort=0 velocity=0 -> lower=-1.5708 upper=3.14159 effort=52 velocity=6.0
- joint left_shoulder_Z: limit lower=-3.14159 upper=3.14159 effort=92 velocity=0 -> lower=-3.14159 upper=3.14159 effort=92 velocity=17.6; origin xyz=0.00805 -0.0728 -0.2037 rpy=0 -0 0 -> xyz=0.008 -0.075 -0.21 rpy=0 -0 0
- joint left_wrist_X: axis -1 0 0 -> 1 0 0; limit lower=-0.785398 upper=0.785398 effort=0 velocity=0 -> lower=-0.785398 upper=0.785398 effort=100 velocity=6.0
- joint left_wrist_Z: limit lower=-1.5708 upper=1.5708 effort=185 velocity=0 -> lower=-1.5708 upper=1.5708 effort=185 velocity=25.0; origin xyz=0 -0.27965 0 rpy=0 -0 0 -> xyz=0 -0.287 0 rpy=0 -0 0
- joint middle_cervical_X: limit lower=-1.5708 upper=1.5708 effort=0 velocity=0 -> lower=-1.5708 upper=1.5708 effort=100 velocity=8.7
- joint middle_cervical_Y: limit lower=-1.5708 upper=1.5708 effort=0 velocity=0 -> lower=-1.5708 upper=1.5708 effort=100 velocity=8.7
- joint middle_cervical_Z: limit lower=-1.5708 upper=1.5708 effort=0 velocity=0 -> lower=-1.5708 upper=1.5708 effort=100 velocity=8.7; origin xyz=0 0.330225 0 rpy=0 -0 0 -> xyz=0 0.25 0 rpy=0 -0 0
- joint middle_lumbar_X: limit lower=-0.785398 upper=0.785398 effort=159 velocity=0 -> lower=-0.785398 upper=0.785398 effort=160 velocity=5.2
- joint middle_lumbar_Z: limit lower=-3.14159 upper=0.785398 effort=243 velocity=0 -> lower=-0.785398 upper=3.14159 effort=190 velocity=5.2
- joint middle_thoracic_X: limit lower=-1.0472 upper=1.0472 effort=159 velocity=0 -> lower=-1.0472 upper=1.0472 effort=190 velocity=5.2
- joint middle_thoracic_Y: limit lower=-1.0472 upper=1.0472 effort=159 velocity=0 -> lower=-1.0472 upper=1.0472 effort=185 velocity=2.0
- joint middle_thoracic_Z: limit lower=-1.0472 upper=0.392699 effort=159 velocity=0 -> lower=-0.392699 upper=1.0472 effort=190 velocity=5.2; origin xyz=0 0.149275 0 rpy=0 -0 0 -> xyz=0 0.223 0 rpy=0 -0 0
- joint right_ankle_X: limit lower=-0.523598333 upper=0.785398 effort=20 velocity=0 -> lower=-0.523598333 upper=0.785398 effort=20 velocity=6.0
- joint right_ankle_Z: limit lower=-1.570795 upper=0.7853975 effort=126 velocity=0 -> lower=-1.570795 upper=0.7853975 effort=126 velocity=12.7; origin xyz=0 -0.42805 0 rpy=0 -0 0 -> xyz=0 -0.44 0 rpy=0 -0 0
- joint right_clavicle_joint_X: limit lower=-0.392699 upper=1.0472 effort=0 velocity=0 -> lower=-0.349066 upper=1.0472 effort=100 velocity=14.0; origin xyz=0 0.330225 0 rpy=0 -0 0 -> xyz=0 0.176 0 rpy=0 -0 0
- joint right_elbow_Y: limit lower=-0.2 upper=3.14159 effort=15 velocity=0 -> lower=-0.349066 upper=3.14159 effort=15 velocity=6.0
- joint right_elbow_Z: limit lower=0 upper=2.617991667 effort=77 velocity=0 -> lower=0 upper=2.617991667 effort=77 velocity=19.9; origin xyz=0 -0.2737 0 rpy=0 -0 0 -> xyz=0 -0.276 0 rpy=0 -0 0
- joint right_hip_X: axis 1 0 0 -> -1 0 0; limit lower=-1.570795 upper=1.047196667 effort=190 velocity=0 -> lower=-1.047196667 upper=1.570795 effort=120 velocity=6.0
- joint right_hip_Y: limit lower=-1.570795 upper=1.047196667 effort=190 velocity=0 -> lower=-1.570795 upper=1.047196667 effort=60 velocity=6.0
- joint right_hip_Z: limit lower=-1.047196667 upper=3.14159 effort=190 velocity=0 -> lower=-1.047196667 upper=3.14159 effort=185 velocity=12.0; origin xyz=0.053375 -0.0749 0.079975 rpy=0 -0 0 -> xyz=0.023 -0.1 0.082 rpy=0 -0 0
- joint right_shoulder_X: limit lower=-1.0472 upper=3.14159 effort=71 velocity=0 -> lower=-1.0472 upper=3.14159 effort=71 velocity=6.0
- joint right_shoulder_Y: axis 0 -1 0 -> 0 1 0; limit lower=-1.5708 upper=3.14159 effort=0 velocity=0 -> lower=-1.5708 upper=3.14159 effort=52 velocity=6.0
- joint right_shoulder_Z: limit lower=-3.14159 upper=3.14159 effort=0 velocity=0 -> lower=-3.14159 upper=3.14159 effort=92 velocity=17.6; origin xyz=0.00805 -0.0728 0.2037 rpy=0 -0 0 -> xyz=0.008 -0.075 0.21 rpy=0 -0 0
- joint right_wrist_X: axis 1 0 0 -> -1 0 0; limit lower=-0.785398 upper=0.785398 effort=0 velocity=0 -> lower=-0.785398 upper=0.785398 effort=100 velocity=6.0
- joint right_wrist_Z: limit lower=-1.5708 upper=1.5708 effort=185 velocity=0 -> lower=-1.5708 upper=1.5708 effort=100 velocity=25.0; origin xyz=0 -0.27965 0 rpy=0 -0 0 -> xyz=0 -0.287 0 rpy=0 -0 0
